Commit message: теперь параметр родительского link'а передается с помощью параметра `parent` езде

File: maddrive_urdf_tools/urdf/macros/damping_wheels.urdf.xacro (robot description, xacro)
@@ -7,5 +7,5 @@
 	<xacro:include filename="$(find maddrive_urdf_tools)/urdf/macros/wheels.urdf.xacro" />
 	<!-- WHEEL SPEED -->
-	<xacro:macro name="speed_wheel" params="name base_name xyz ">
+	<xacro:macro name="speed_wheel" params="name parent xyz ">
 		<base_wheel name="wheel_${name}" />
 		<gazebo reference="${name}_spring_joint">
@@ -16,5 +16,5 @@
 		<joint name="${name}_spring_joint" type="prismatic">
 			<limit lower="-0.1" upper="0.1" effort="0" velocity="0" />
-			<parent link="${base_name}" />
+			<parent link="${parent}" />
 			<child link="spring1_${name}" />
 			<dynamics damping="0.0" friction="0.0" />
@@ -33,5 +33,5 @@
 	</xacro:macro>
 	<!-- WHEEL STEER -->
-	<xacro:macro name="steer_wheel" params="name base_name xyz">
+	<xacro:macro name="steer_wheel" params="name parent xyz">
 		<base_wheel name="wheel_${name}" />
 		<gazebo reference="${name}_spring_joint">
@@ -42,5 +42,5 @@
 		<joint name="${name}_spring_joint" type="prismatic">
 			<limit lower="-0.1" upper="0.1" effort="0" velocity="0" />
-			<parent link="${base_name}" />
+			<parent link="${parent}" />
 			<child link="spring2_${name}" />
 			<dynamics damping="0.0" friction="0.0" />

File: maddrive_urdf_tools/urdf/macros/elp_stereo.urdf.xacro (robot description, xacro)
@@ -7,5 +7,5 @@
 	<xacro:property name="elp_camera_length" value="0.015" />
 	<xacro:property name="elp_camera_mass_kg" value="0.15" />
-	<xacro:macro name="elp_stereo" params="name base_link_name xyz rpy">
+	<xacro:macro name="elp_stereo" params="name parent xyz rpy">
 		<link name="${name}_link">
 			<visual>
@@ -28,5 +28,5 @@
 		</link>
 		<joint name="base_${name}_camera_joint" type="fixed">
-			<parent link="${base_link_name}" />
+			<parent link="${parent}" />
 			<child link="${name}_link" />
 			<origin xyz="${xyz}" rpy="${rpy}" />

File: maddrive_urdf_tools/urdf/macros/lidar.urdf.xacro (robot description, xacro)
@@ -4,5 +4,5 @@
     <xacro:property name="lidar_height" value="0.02" />
     <xacro:property name="lidar_radius" value="0.04" />
-    <xacro:macro name="simple_lidar" params="name base_name place_height">
+    <xacro:macro name="simple_lidar" params="name parent place_height">
         <link name="${name}">
             <cylinder_inertial r="${lidar_radius}" h="${lidar_height}" mass="${lidar_mass}">
@@ -25,5 +25,5 @@
             <axis xyz="0 1 0" />
             <origin xyz="0 0 ${place_height}" rpy="0 0 0" />
-            <parent link="${base_name}" />
+            <parent link="${parent}" />
             <child link="lidar_link" />
         </joint>

File: maddrive_urdf_tools/urdf/macros/realsense.urdf.xacro (robot description, xacro)
@@ -13,5 +13,5 @@
     <xacro:macro
         name="realsense_435"
-        params="name base_link_name xyz rpy">
+        params="name parent xyz rpy">
         <link name="${name}_link">
             <visual>
@@ -34,5 +34,5 @@
         </link>
         <joint name="base_${name}_camera_joint" type="fixed">
-            <parent link="${base_link_name}" />
+            <parent link="${parent}" />
             <child link="${name}_link" />
             <origin xyz="${xyz}" rpy="${rpy}" />
