Commit message: добавил макросы для отсутсвия модели столкновения и инерции

File: maddrive_urdf_tools/urdf/macros/common.urdf.xacro (robot description, xacro)
@@ -6,3 +6,7 @@
     <xacro:macro name="null_visual" >
     </xacro:macro>
+    <xacro:macro name="null_collision" >
+    </xacro:macro>
+    <xacro:macro name="null_inertia" >
+    </xacro:macro>
 </robot>
