Commit message: исправил дальность у лидара c64

File: maddrive_urdf_tools/urdf/macros/sector_lidar.urdf.xacro (robot description, xacro)
@@ -22,6 +22,6 @@
     <xacro:property name="c64_lidar_vertical_min_angle" value="-0.436332" />
     <xacro:property name="c64_lidar_vertical_max_angle" value="0.261799" />
-    <xacro:property name="c64_lidar_range_min" value="0.2" />
-    <xacro:property name="c64_lidar_range_max" value="20" />
+    <xacro:property name="c64_lidar_range_min" value="0.5" />
+    <xacro:property name="c64_lidar_range_max" value="100" />
     <xacro:macro name="sector_lidar" params="model parent origin_xyz origin_rpy">
         <joint name="${model}_lidar_joint" type="fixed">

Commit message: renamed the lidar data output topic for further message conversion + all conversion package + change a colisional wheel-ball model (to reduce slippage)

File: maddrive_urdf_tools/urdf/macros/sector_lidar.urdf.xacro (robot description, xacro)
@@ -81,6 +81,5 @@
             <material>Gazebo/Blue</material>
             <sensor name="${prefix}_lslidar_${model}_lidar_sensor" type="ray">
-                <pose>0 0 0.0 0 0 0</pose>
-                <visualize>true</visualize>
+                <visualize>false</visualize>
                 <ray>
                     <scan>
@@ -130,5 +129,5 @@
                     <robotNamespace>/</robotNamespace>
                     <frameName>${prefix}_lslidar_${model}_lidar_link</frameName>
-                    <topicName>${prefix}_lslidar_${model}_lidar_point_cloud</topicName>
+                    <topicName>${prefix}_lslidar_${model}_lidar_point_cloud_pcl1</topicName>
                     <gaussianNoise>0.01</gaussianNoise>
                     <hokuyoMinIntensity>101</hokuyoMinIntensity>

File: maddrive_urdf_tools/urdf/macros/wheels.urdf.xacro (robot description, xacro)
@@ -15,5 +15,6 @@
 				<origin xyz="0 0 0" rpy="${pi/2} 0 0" />
 				<geometry>
-					<cylinder length="${wheel_width}" radius="${wheel_radius}" />
+					<sphere radius="${wheel_radius}" />
+					<!-- <cylinder length="${wheel_width}" radius="${wheel_radius}" /> -->
 				</geometry>
 			</collision>
