Commit message: местами немного подровнял файлы

File: maddrive_urdf_tools/urdf/macros/camera.urdf.xacro (robot description, xacro)
@@ -35,11 +35,7 @@
 		</joint>
 		<gazebo reference="${direction}_${position}_cam_frame">
-			<material>
-			Gazebo/Orange
-		</material>
+			<material>Gazebo/Orange</material>
 			<sensor type="camera" name="${direction}_${position}_cam">
-				<update_rate>
-				30.0
-			</update_rate>
+				<update_rate>30.0</update_rate>
 				<camera name="${direction}_${position}_cam">
 					<horizontal_fov>${fov}</horizontal_fov>

File: maddrive_urdf_tools/urdf/macros/damping_wheels.urdf.xacro (robot description, xacro)
@@ -6,5 +6,5 @@
 	<xacro:include filename="$(find maddrive_urdf_tools)/urdf/macros/common.urdf.xacro" />
 	<xacro:include filename="$(find maddrive_urdf_tools)/urdf/macros/wheels.urdf.xacro" />
-	<!-- XACRO SPEED -->
+	<!-- WHEEL SPEED -->
 	<xacro:macro name="speed_wheel" params="name base_name xyz ">
 		<base_wheel name="wheel_${name}" />
@@ -32,5 +32,5 @@
 		</joint>
 	</xacro:macro>
-	<!-- XACRO STEER -->
+	<!-- WHEEL STEER -->
 	<xacro:macro name="steer_wheel" params="name base_name xyz">
 		<base_wheel name="wheel_${name}" />
@@ -51,5 +51,9 @@
 		</link>
 		<joint name="${name}_steer_joint" type="revolute">
-			<limit lower="${-wheel_turn_limit}" upper="${wheel_turn_limit}" effort="1000" velocity="0" />
+			<limit
+				lower="${-wheel_turn_limit}"
+				upper="${wheel_turn_limit}"
+				effort="1000"
+				velocity="0" />
 			<parent link="spring2_${name}" />
 			<child link="steer_${name}" />

File: maddrive_urdf_tools/urdf/macros/elp_stereo.urdf.xacro (robot description, xacro)
@@ -3,19 +3,9 @@
 	<xacro:include filename="$(find maddrive_urdf_tools)/urdf/macros/inertia.urdf.xacro" />
 	<xacro:include filename="$(find maddrive_urdf_tools)/urdf/macros/common.urdf.xacro" />
-	<xacro:property
-			name="elp_camera_width"
-			value="0.1" />
-	<xacro:property
-			name="elp_camera_height"
-			value="0.03" />
-	<xacro:property
-			name="elp_camera_length"
-			value="0.015" />
-	<xacro:property
-			name="elp_camera_mass_kg"
-			value="0.15" />
-	<xacro:macro
-			name="elp_stereo"
-			params="name base_link_name xyz rpy">
+	<xacro:property name="elp_camera_width" value="0.1" />
+	<xacro:property name="elp_camera_height" value="0.03" />
+	<xacro:property name="elp_camera_length" value="0.015" />
+	<xacro:property name="elp_camera_mass_kg" value="0.15" />
+	<xacro:macro name="elp_stereo" params="name base_link_name xyz rpy">
 		<link name="${name}_link">
 			<visual>
@@ -30,37 +20,25 @@
 			</collision>
 			<xacro:box_inertia
-					width="${elp_camera_width}"
-					length="${elp_camera_length}"
-					height="${elp_camera_height}"
-					mass="${elp_camera_mass_kg}">
-				<origin
-						xyz="0 0 0"
-						rpy="0 0 0" />
+				width="${elp_camera_width}"
+				length="${elp_camera_length}"
+				height="${elp_camera_height}"
+				mass="${elp_camera_mass_kg}">
+				<origin xyz="0 0 0" rpy="0 0 0" />
 			</xacro:box_inertia>
 		</link>
-		<joint
-				name="base_${name}_camera_joint"
-				type="fixed">
+		<joint name="base_${name}_camera_joint" type="fixed">
 			<parent link="${base_link_name}" />
 			<child link="${name}_link" />
-			<origin
-					xyz="${xyz}"
-					rpy="${rpy}" />
+			<origin xyz="${xyz}" rpy="${rpy}" />
 		</joint>
 		<link name="${name}_optical_frame" />
-		<joint
-				name="${name}_camera_optical_joint"
-				type="fixed">
+		<joint name="${name}_camera_optical_joint" type="fixed">
 			<parent link="${name}_link" />
 			<child link="${name}_optical_frame" />
-			<origin
-					xyz="0 0 0"
-					rpy="${-pi/2} 0 ${-pi/2}" />
+			<origin xyz="0 0 0" rpy="${-pi/2} 0 ${-pi/2}" />
 		</joint>
 		<gazebo reference="${name}_link">
 			<material>Gazebo/Green</material>
-			<sensor
-					name="${name}"
-					type="depth">
+			<sensor name="${name}" type="depth">
 				<update_rate>25</update_rate>
 				<camera>
@@ -76,7 +54,5 @@
 					</clip>
 				</camera>
-				<plugin
-						name="camera_plugin"
-						filename="libgazebo_ros_openni_kinect.so">
+				<plugin name="camera_plugin" filename="libgazebo_ros_openni_kinect.so">
 					<baseline>0.06</baseline>
 					<alwaysOn>true</alwaysOn>

File: maddrive_urdf_tools/urdf/macros/inertia.urdf.xacro (robot description, xacro)
@@ -1,44 +1,45 @@
 <?xml version="1.0"?>
 <robot xmlns:xacro="http://www.ros.org/wiki/xacro">
-	<xacro:macro name="null_inertial">
+	<xacro:macro
+		name="null_inertial">
 		<inertial>
 			<mass value="0.1" />
 			<inertia
-					ixx="0.01"
-					ixy="0"
-					ixz="0"
-					iyy="0.01"
-					iyz="0"
-					izz="0.01" />
+				ixx="0.01"
+				ixy="0"
+				ixz="0"
+				iyy="0.01"
+				iyz="0"
+				izz="0.01" />
 		</inertial>
 	</xacro:macro>
 	<xacro:macro
-			name="box_inertia"
-			params="width length height mass *origin">
+		name="box_inertia"
+		params="width length height mass *origin">
 		<inertial>
 			<xacro:insert_block name="origin" />
 			<mass value="${mass}" />
 			<inertia
-					ixx="${mass * (width * width + height * height) / 12}"
-					ixy="0"
-					ixz="0"
-					iyy="${mass * (length * length + height * height) / 12}"
-					iyz="0"
-					izz="${mass * (width * width + length * length) / 12}" />
+				ixx="${mass * (width * width + height * height) / 12}"
+				ixy="0"
+				ixz="0"
+				iyy="${mass * (length * length + height * height) / 12}"
+				iyz="0"
+				izz="${mass * (width * width + length * length) / 12}" />
 		</inertial>
 	</xacro:macro>
 	<xacro:macro
-			name="cylinder_inertia"
-			params="r h mass *origin">
+		name="cylinder_inertia"
+		params="r h mass *origin">
 		<inertial>
 			<xacro:insert_block name="origin" />
 			<mass value="${mass}" />
 			<inertia
-					ixx="${mass / 12 * (3 * r * r + h * h)}"
-					ixy="0.0"
-					ixz="0.0"
-					iyy="${mass / 12 * (3 * r * r + h * h)}"
-					iyz="0.0"
-					izz="${mass / 2 * r * r}" />
+				ixx="${mass / 12 * (3 * r * r + h * h)}"
+				ixy="0.0"
+				ixz="0.0"
+				iyy="${mass / 12 * (3 * r * r + h * h)}"
+				iyz="0.0"
+				izz="${mass / 2 * r * r}" />
 		</inertial>
 	</xacro:macro>

File: maddrive_urdf_tools/urdf/macros/lidar.urdf.xacro (robot description, xacro)
@@ -1,64 +1,63 @@
 <?xml version="1.0"?>
 <robot xmlns:xacro="http://www.ros.org/wiki/xacro">
-  <xacro:property name="lidar_mass" value="0.1" />
-  <xacro:property name="lidar_height" value="0.02" />
-  <xacro:property name="lidar_radius" value="0.04" />
-  <xacro:macro name="simple_lidar" params="name base_name place_height">
-    <link name="${name}">
-      <cylinder_inertial r="${lidar_radius}" h="${lidar_height}" mass="${lidar_mass}">
-        <origin xyz="0 0 0" rpy="0 0 0" />
-      </cylinder_inertial>
-      <collision>
-        <origin xyz="0 0 0" rpy="0 0 0" />
-        <geometry>
-          <cylinder length="${lidar_height}" radius="${lidar_radius}" />
-        </geometry>
-      </collision>
-      <visual>
-        <origin xyz="0 0 0" rpy="0 0 0" />
-        <geometry>
-          <cylinder length="${lidar_height}" radius="${lidar_radius}" />
-        </geometry>
-      </visual>
-    </link>
-    <joint name="lidar_joint" type="fixed">
-      <axis xyz="0 1 0" />
-      <origin xyz="0 0 ${place_height}" rpy="0 0 0" />
-      <parent link="${base_name}" />
-      <child link="lidar_link" />
-    </joint>
-    <!-- GAZEBO -->
-    <gazebo reference="lidar_link">
-      <material>Gazebo/Red</material>
-      <sensor type="ray" name="head_hokuyo_sensor">
-        <pose>0 0 0 0 0 0</pose>
-        <visualize>false</visualize>
-        <update_rate>40</update_rate>
-        <ray>
-          <scan>
-            <horizontal>
-              <samples>720</samples>
-              <resolution>1</resolution>
-              <min_angle>-3.14</min_angle>
-              <max_angle>3.14</max_angle>
-            </horizontal>
-          </scan>
-          <range>
-            <min>0.10</min>
-            <max>30.0</max>
-            <resolution>0.01</resolution>
-          </range>
-          <noise>
-            <type>gaussian</type>
-            <mean>0.0</mean>
-            <stddev>0.01</stddev>
-          </noise>
-        </ray>
-        <plugin name="gazebo_ros_head_hokuyo_controller" filename="libgazebo_ros_laser.so">
-          <topicName>/scan</topicName>
-          <frameName>lidar_link</frameName>
-        </plugin>
-      </sensor>
-    </gazebo>
-  </xacro:macro>
+    <xacro:property name="lidar_mass" value="0.1" />
+    <xacro:property name="lidar_height" value="0.02" />
+    <xacro:property name="lidar_radius" value="0.04" />
+    <xacro:macro name="simple_lidar" params="name base_name place_height">
+        <link name="${name}">
+            <cylinder_inertial r="${lidar_radius}" h="${lidar_height}" mass="${lidar_mass}">
+                <origin xyz="0 0 0" rpy="0 0 0" />
+            </cylinder_inertial>
+            <collision>
+                <origin xyz="0 0 0" rpy="0 0 0" />
+                <geometry>
+                    <cylinder length="${lidar_height}" radius="${lidar_radius}" />
+                </geometry>
+            </collision>
+            <visual>
+                <origin xyz="0 0 0" rpy="0 0 0" />
+                <geometry>
+                    <cylinder length="${lidar_height}" radius="${lidar_radius}" />
+                </geometry>
+            </visual>
+        </link>
+        <joint name="lidar_joint" type="fixed">
+            <axis xyz="0 1 0" />
+            <origin xyz="0 0 ${place_height}" rpy="0 0 0" />
+            <parent link="${base_name}" />
+            <child link="lidar_link" />
+        </joint>
+        <gazebo reference="lidar_link">
+            <material>Gazebo/Red</material>
+            <sensor name="head_hokuyo_sensor" type="ray">
+                <pose>0 0 0 0 0 0</pose>
+                <visualize>false</visualize>
+                <update_rate>40</update_rate>
+                <ray>
+                    <scan>
+                        <horizontal>
+                            <samples>720</samples>
+                            <resolution>1</resolution>
+                            <min_angle>-3.14</min_angle>
+                            <max_angle>3.14</max_angle>
+                        </horizontal>
+                    </scan>
+                    <range>
+                        <min>0.10</min>
+                        <max>30.0</max>
+                        <resolution>0.01</resolution>
+                    </range>
+                    <noise>
+                        <type>gaussian</type>
+                        <mean>0.0</mean>
+                        <stddev>0.01</stddev>
+                    </noise>
+                </ray>
+                <plugin name="gazebo_ros_head_hokuyo_controller" filename="libgazebo_ros_laser.so">
+                    <topicName>/scan</topicName>
+                    <frameName>lidar_link</frameName>
+                </plugin>
+            </sensor>
+        </gazebo>
+    </xacro:macro>
 </robot>

File: maddrive_urdf_tools/urdf/macros/realsense.urdf.xacro (robot description, xacro)
@@ -3,28 +3,15 @@
     <xacro:include filename="$(find maddrive_urdf_tools)/urdf/macros/inertia.urdf.xacro" />
     <xacro:include filename="$(find maddrive_urdf_tools)/urdf/macros/common.urdf.xacro" />
-    <xacro:property
-            name="rs_camera_width"
-            value="0.09" />
-    <xacro:property
-            name="rs_camera_height"
-            value="0.025" />
-    <xacro:property
-            name="rs_camera_length"
-            value="0.025" />
-    <xacro:property
-            name="rs_camera_mass_kg"
-            value="0.320" />
-    <xacro:property
-            name="rs_imu_height"
-            value="0.01" />
-    <xacro:property
-            name="rs_imu_width"
-            value="0.01" />
-    <xacro:property
-            name="rs_imu_length"
-            value="0.01" />
+    <xacro:property name="rs_camera_width" value="0.09" />
+    <xacro:property name="rs_camera_height" value="0.025" />
+    <xacro:property name="rs_camera_length" value="0.025" />
+    <xacro:property name="rs_camera_mass_kg" value="0.320" />
+    <xacro:property name="rs_imu_height" value="0.01" />
+    <xacro:property name="rs_imu_width" value="0.01" />
+    <xacro:property name="rs_imu_length" value="0.01" />
+    <!-- DEPTH CAMERA -->
     <xacro:macro
-            name="realsense_435"
-            params="name base_link_name xyz rpy">
+        name="realsense_435"
+        params="name base_link_name xyz rpy">
         <link name="${name}_link">
             <visual>
@@ -39,37 +26,25 @@
             </collision>
             <xacro:box_inertia
-                    width="${rs_camera_width}"
-                    length="${rs_camera_length}"
-                    height="${rs_camera_height}"
-                    mass="${rs_camera_mass_kg}">
-                <origin
-                        xyz="0 0 0"
-                        rpy="0 0 0" />
+                width="${rs_camera_width}"
+                length="${rs_camera_length}"
+                height="${rs_camera_height}"
+                mass="${rs_camera_mass_kg}">
+                <origin xyz="0 0 0" rpy="0 0 0" />
             </xacro:box_inertia>
         </link>
-        <joint
-                name="base_${name}_camera_joint"
-                type="fixed">
+        <joint name="base_${name}_camera_joint" type="fixed">
             <parent link="${base_link_name}" />
             <child link="${name}_link" />
-            <origin
-                    xyz="${xyz}"
-                    rpy="${rpy}" />
+            <origin xyz="${xyz}" rpy="${rpy}" />
         </joint>
         <link name="${name}_optical_frame" />
-        <joint
-                name="${name}_camera_optical_joint"
-                type="fixed">
+        <joint name="${name}_camera_optical_joint" type="fixed">
             <parent link="${name}_link" />
             <child link="${name}_optical_frame" />
-            <origin
-                    xyz="0 0 0"
-                    rpy="${-pi/2} 0 ${-pi/2}" />
+            <origin xyz="0 0 0" rpy="${-pi/2} 0 ${-pi/2}" />
         </joint>
         <gazebo reference="${name}_link">
             <material>Gazebo/Black</material>
-            <sensor
-                    name="${name}"
-                    type="depth">
+            <sensor name="${name}" type="depth">
                 <update_rate>20</update_rate>
                 <camera>
@@ -85,7 +60,5 @@
                     </clip>
                 </camera>
-                <plugin
-                        name="camera_plugin"
-                        filename="libgazebo_ros_openni_kinect.so">
+                <plugin name="camera_plugin" filename="libgazebo_ros_openni_kinect.so">
                     <baseline>0.2</baseline>
                     <alwaysOn>true</alwaysOn>
@@ -127,26 +100,18 @@
             <xacro:null_inertial />
         </link>
-        <joint
-                name="${name}_camera_imu_joint"
-                type="fixed">
+        <joint name="${name}_camera_imu_joint" type="fixed">
             <parent link="${name}_link" />
             <child link="${name}_imu_link" />
-            <origin
-                    xyz="0 0 0"
-                    rpy="0 0 0" />
+            <origin xyz="0 0 0" rpy="0 0 0" />
         </joint>
         <gazebo reference="${name}_imu_link">
             <material>Gazebo/Red</material>
             <gravity>true</gravity>
-            <sensor
-                    name="imu_sensor"
-                    type="imu">
+            <sensor name="imu_sensor" type="imu">
                 <always_on>true</always_on>
                 <update_rate>100</update_rate>
                 <visualize>true</visualize>
                 <topic>__default_topic__</topic>
-                <plugin
-                        filename="libgazebo_ros_imu_sensor.so"
-                        name="imu_plugin">
+                <plugin filename="libgazebo_ros_imu_sensor.so" name="imu_plugin">
                     <topicName>/${name}/imu/</topicName>
                     <bodyName>${name}_imu_link</bodyName>

File: maddrive_urdf_tools/urdf/macros/wheels.urdf.xacro (robot description, xacro)
@@ -4,5 +4,5 @@
 	<xacro:include filename="$(find maddrive_urdf_tools)/urdf/macros/inertia.urdf.xacro" />
 	<xacro:include filename="$(find maddrive_urdf_tools)/urdf/macros/common.urdf.xacro" />
-	<!-- XACRO WHEEL -->
+	<!-- BASE WHEEL -->
 	<xacro:macro name="base_wheel" params="name">
 		<link name="${name}">
@@ -27,5 +27,5 @@
 		</gazebo>
 	</xacro:macro>
-	<!-- XACRO SPEED -->
+	<!-- SPEED WHEEL -->
 	<xacro:macro name="speed_wheel" params="name base_name xyz ">
 		<xacro:base_wheel name="wheel_${name}" />
@@ -38,5 +38,5 @@
 		</joint>
 	</xacro:macro>
-	<!-- XACRO STEER -->
+	<!-- STEER WHEEL -->
 	<xacro:macro name="steer_wheel" params="name base_name xyz steer_limit">
 		<xacro:base_wheel name="wheel_${name}" />

Commit message: add sphere inertia urdf-macro; replace "inertial" to "inertia" to reduse confusion

File: maddrive_urdf_tools/urdf/macros/camera.urdf.xacro (robot description, xacro)
@@ -18,5 +18,5 @@
 				</geometry>
 			</collision>
-			<null_inertial />
+			<null_inertia />
 		</link>
 	</xacro:macro>

File: maddrive_urdf_tools/urdf/macros/common.urdf.xacro (robot description, xacro)
@@ -5,8 +5,30 @@
     <xacro:property name="degrees_180" value="${pi}" />
     <xacro:macro name="null_visual" >
+        <visual>
+			<origin xyz="0 0 0" rpy="0 0 0" />
+			<geometry>
+				<box size="0 0 0" />
+			</geometry>
+		</visual>
     </xacro:macro>
     <xacro:macro name="null_collision" >
+        <collision name="base_collision">
+			<origin xyz="0 0 0" rpy="0 0 0" />
+			<geometry>
+				<box size="0 0 0" />
+			</geometry>
+		</collision>
     </xacro:macro>
-    <xacro:macro name="null_inertia" >
+	<xacro:macro name="null_inertia" >
+        <inertial>
+			<mass value="0.01" />
+			<inertia
+				ixx="0.01"
+				ixy="0.01"
+				ixz="0.01"
+				iyy="0.01"
+				iyz="0.01"
+				izz="0.01" />
+		</inertial>
     </xacro:macro>
 </robot>

File: maddrive_urdf_tools/urdf/macros/damping_wheels.urdf.xacro (robot description, xacro)
@@ -22,5 +22,5 @@
 		</joint>
 		<link name="spring1_${name}">
-			<null_inertial />
+			<null_inertia />
 		</link>
 		<joint name="${name}_speed_joint" type="continuous">
@@ -48,5 +48,5 @@
 		</joint>
 		<link name="spring2_${name}">
-			<null_inertial />
+			<null_inertia />
 		</link>
 		<joint name="${name}_steer_joint" type="revolute">
@@ -62,5 +62,5 @@
 		</joint>
 		<link name="steer_${name}">
-			<null_inertial />
+			<null_inertia />
 		</link>
 		<joint name="${name}_speed_joint" type="continuous">

File: maddrive_urdf_tools/urdf/macros/inertia.urdf.xacro (robot description, xacro)
@@ -1,17 +1,4 @@
 <?xml version="1.0"?>
 <robot xmlns:xacro="http://www.ros.org/wiki/xacro">
-	<xacro:macro
-		name="null_inertial">
-		<inertial>
-			<mass value="0.1" />
-			<inertia
-				ixx="0.01"
-				ixy="0"
-				ixz="0"
-				iyy="0.01"
-				iyz="0"
-				izz="0.01" />
-		</inertial>
-	</xacro:macro>
 	<xacro:macro
 		name="box_inertia"
@@ -44,3 +31,18 @@
 		</inertial>
 	</xacro:macro>
+	<xacro:macro
+		name="sphere_inertia"
+		params="r mass *origin">
+		<inertial>
+			<xacro:insert_block name="origin" />
+			<mass value="${mass}"/>
+			<inertia
+				ixx="${2 * mass * r * r / 5}"
+				ixy="0.0"
+				ixz="0.0"
+				iyy="${2 * mass * r * r / 5}"
+				iyz="0.0"
+				izz="${2 * mass * r * r / 5}"/>
+		</inertial>
+	</xacro:macro>
 </robot>

File: maddrive_urdf_tools/urdf/macros/lidar.urdf.xacro (robot description, xacro)
@@ -23,8 +23,7 @@
         </link>
         <joint name="lidar_joint" type="fixed">
-            <axis xyz="0 1 0" />
-            <origin xyz="0 0 ${place_height}" rpy="0 0 0" />
             <parent link="${parent}" />
             <child link="lidar_link" />
+            <origin xyz="0 0 ${place_height}" rpy="0 0 0" />
         </joint>
         <gazebo reference="lidar_link">

File: maddrive_urdf_tools/urdf/macros/realsense.urdf.xacro (robot description, xacro)
@@ -158,5 +158,5 @@
                 </geometry>
             </collision>
-            <xacro:null_inertial />
+            <xacro:null_inertia />
         </link>
         <gazebo reference="${prefix}_rs_${model}_camera_imu_link">

File: maddrive_urdf_tools/urdf/macros/wheels.urdf.xacro (robot description, xacro)
@@ -51,6 +51,9 @@
 		</joint>
 		<link name="${prefix}_steer_link">
-			<xacro:null_inertial />
+			<xacro:null_visual />
+			<xacro:null_collision />
+			<xacro:null_inertia />
 		</link>
+		<gazebo reference="${prefix}_steer_link" />
 		<joint name="${prefix}_wheel_joint" type="continuous">
 			<parent link="${prefix}_steer_link" />
