Commit message: a description of mechanisms has been added to the description of the wheels for the possibility of using plugins that require it (four_wheel_steering, for example); an explicit indication of object parameters has been added to the inertia macro

File: maddrive_urdf_tools/urdf/macros/inertia.urdf.xacro (robot description, xacro)
@@ -18,30 +18,30 @@
 	<xacro:macro
 		name="cylinder_inertia"
-		params="r h mass *origin">
+		params="radius length mass *origin">
 		<inertial>
 			<xacro:insert_block name="origin" />
 			<mass value="${mass}" />
 			<inertia
-				ixx="${mass / 12 * (3 * r * r + h * h)}"
+				ixx="${mass / 12 * (3 * radius * radius + length * length)}"
 				ixy="0.0"
 				ixz="0.0"
-				iyy="${mass / 12 * (3 * r * r + h * h)}"
+				iyy="${mass / 12 * (3 * radius * radius + length * length)}"
 				iyz="0.0"
-				izz="${mass / 2 * r * r}" />
+				izz="${mass / 2 * radius * radius}" />
 		</inertial>
 	</xacro:macro>
 	<xacro:macro
 		name="sphere_inertia"
-		params="r mass *origin">
+		params="radius mass *origin">
 		<inertial>
 			<xacro:insert_block name="origin" />
 			<mass value="${mass}"/>
 			<inertia
-				ixx="${2 * mass * r * r / 5}"
+				ixx="${2 * mass * radius * radius / 5}"
 				ixy="0.0"
 				ixz="0.0"
-				iyy="${2 * mass * r * r / 5}"
+				iyy="${2 * mass * radius * radius / 5}"
 				iyz="0.0"
-				izz="${2 * mass * r * r / 5}"/>
+				izz="${2 * mass * radius * radius / 5}"/>
 		</inertial>
 	</xacro:macro>

File: maddrive_urdf_tools/urdf/macros/lidar.urdf.xacro (robot description, xacro)
@@ -6,5 +6,8 @@
     <xacro:macro name="simple_lidar" params="name parent place_height">
         <link name="${name}">
-            <cylinder_inertial r="${lidar_radius}" h="${lidar_height}" mass="${lidar_mass}">
+            <cylinder_inertial
+                radius="${lidar_radius}"
+                length="${lidar_height}"
+                mass="${lidar_mass}">
                 <origin xyz="0 0 0" rpy="0 0 0" />
             </cylinder_inertial>

File: maddrive_urdf_tools/urdf/macros/sector_lidar.urdf.xacro (robot description, xacro)
@@ -63,6 +63,6 @@
             <xacro:if value="${model == 'c16'}">
                 <xacro:cylinder_inertia
-                    r="${c16_radius}"
-                    h="${c16_height}"
+                    radius="${c16_radius}"
+                    length="${c16_height}"
                     mass="${c16_mass_kg}">
                     <origin xyz="0 0 0" rpy="0 0 0" />
@@ -71,6 +71,6 @@
             <xacro:if value="${model == 'c64'}">
                 <xacro:cylinder_inertia
-                    r="${c64_radius}"
-                    h="${c64_height}"
+                    radius="${c64_radius}"
+                    length="${c64_height}"
                     mass="${c64_mass_kg}">
                     <origin xyz="0 0 0" rpy="0 0 0" />

File: maddrive_urdf_tools/urdf/macros/wheels.urdf.xacro (robot description, xacro)
@@ -19,5 +19,8 @@
 				</geometry>
 			</collision>
-			<xacro:cylinder_inertia r="${wheel_radius}" h="${wheel_width}" mass="${wheel_mass}">
+			<xacro:cylinder_inertia
+				radius="${wheel_radius}"
+				length="${wheel_width}"
+				mass="${wheel_mass}">
 				<origin xyz="0 0 0" rpy="${pi/2} 0 0" />
 			</xacro:cylinder_inertia>
@@ -37,6 +40,16 @@
 			<origin xyz="${origin_xyz}" rpy="0 0 0" />
 			<axis xyz="0 1 0" />
-			<limit effort="0" velocity="0" />
+			<limit effort="100000" velocity="${pi*10}" />
 		</joint>
+		<transmission name="${prefix}_wheel_trans">
+			<type>transmission_interface/SimpleTransmission</type>
+			<joint name="${prefix}_wheel_joint">
+				<hardwareInterface>hardware_interface/VelocityJointInterface</hardwareInterface>
+			</joint>
+			<actuator name="${prefix}_wheel_motor">
+				<hardwareInterface>hardware_interface/VelocityJointInterface</hardwareInterface>
+				<mechanicalReduction>1</mechanicalReduction>
+			</actuator>
+		</transmission>
 		<xacro:base_wheel name="${prefix}_wheel_link" />
 	</xacro:macro>
@@ -48,6 +61,16 @@
 			<origin xyz="${steer_origin_xyz}" rpy="0 0 0" />
 			<axis xyz="0 0 1" />
-			<limit lower="${-steer_limit}" upper="${steer_limit}" effort="0" velocity="0" />
+			<limit lower="${-steer_limit}" upper="${steer_limit}" effort="100000" velocity="${pi*2}" />
 		</joint>
+		<transmission name="${prefix}_steer_trans">
+			<type>transmission_interface/SimpleTransmission</type>
+			<joint name="${prefix}_steer_joint">
+				<hardwareInterface>hardware_interface/PositionJointInterface</hardwareInterface>
+			</joint>
+			<actuator name="${prefix}_steer_motor">
+				<hardwareInterface>hardware_interface/PositionJointInterface</hardwareInterface>
+				<mechanicalReduction>30</mechanicalReduction>
+			</actuator>
+		</transmission>
 		<link name="${prefix}_steer_link">
 			<xacro:null_visual />
@@ -61,6 +84,16 @@
 			<origin xyz="0 0 0" rpy="0 0 0" />
 			<axis xyz="0 1 0" />
-			<limit effort="0" velocity="0" />
+			<limit effort="100000" velocity="${pi*10}" />
 		</joint>
+		<transmission name="${prefix}_wheel_trans">
+			<type>transmission_interface/SimpleTransmission</type>
+			<joint name="${prefix}_wheel_joint">
+				<hardwareInterface>hardware_interface/VelocityJointInterface</hardwareInterface>
+			</joint>
+			<actuator name="${prefix}_wheel_motor">
+				<hardwareInterface>hardware_interface/VelocityJointInterface</hardwareInterface>
+				<mechanicalReduction>1</mechanicalReduction>
+			</actuator>
+		</transmission>
 		<xacro:base_wheel name="${prefix}_wheel_link" />
 	</xacro:macro>
