Commit message: Added ELP camera model

File: maddrive_urdf_tools/urdf/macros/realsense.urdf.xacro (robot description, xacro)
@@ -15,4 +15,13 @@
             name="rs_camera_mass_kg"
             value="0.320" />
+    <xacro:property
+            name="rs_imu_height"
+            value="0.01" />
+    <xacro:property
+            name="rs_imu_width"
+            value="0.01" />
+    <xacro:property
+            name="rs_imu_length"
+            value="0.01" />
     <xacro:macro
             name="realsense_435"
@@ -48,5 +57,5 @@
                     rpy="${rpy}" />
         </joint>
-	    <link name="${name}_optical_frame" />
+        <link name="${name}_optical_frame" />
         <joint
                 name="${name}_camera_optical_joint"
@@ -73,5 +82,5 @@
                     <clip>
                         <near>0.05</near>
-                        <far>20</far>
+                        <far>8</far>
                     </clip>
                 </camera>
@@ -104,5 +113,51 @@
             </sensor>
         </gazebo>
-        <!-- TODO - add IMU -->
+        <!-- IMU -->
+        <link name="${name}_imu_link">
+            <visual>
+                <geometry>
+                    <box size="${rs_imu_length} ${rs_imu_width} ${rs_imu_height}" />
+                </geometry>
+            </visual>
+            <collision>
+                <geometry>
+                    <box size="${rs_imu_length} ${rs_imu_width} ${rs_imu_height}" />
+                </geometry>
+            </collision>
+            <xacro:null_inertial />
+        </link>
+        <joint
+                name="${name}_camera_imu_joint"
+                type="fixed">
+            <parent link="${name}_link" />
+            <child link="${name}_imu_link" />
+            <origin
+                    xyz="0 0 0"
+                    rpy="0 0 0" />
+        </joint>
+        <gazebo reference="${name}_imu_link">
+            <material>Gazebo/Red</material>
+            <gravity>true</gravity>
+            <sensor
+                    name="imu_sensor"
+                    type="imu">
+                <always_on>true</always_on>
+                <update_rate>100</update_rate>
+                <visualize>true</visualize>
+                <topic>__default_topic__</topic>
+                <plugin
+                        filename="libgazebo_ros_imu_sensor.so"
+                        name="imu_plugin">
+                    <topicName>/${name}/imu</topicName>
+                    <bodyName>${name}_imu_link</bodyName>
+                    <updateRateHZ>20.0</updateRateHZ>
+                    <gaussianNoise>0.5</gaussianNoise>
+                    <xyzOffset>0 0 0</xyzOffset>
+                    <rpyOffset>0 0 0</rpyOffset>
+                    <frameName>${name}_imu_link</frameName>
+                </plugin>
+                <pose>0 0 0 0 0 0</pose>
+            </sensor>
+        </gazebo>
     </xacro:macro>
 </robot>

Commit message: fixed realsence macro to use two camera models

File: maddrive_urdf_tools/urdf/macros/realsense.urdf.xacro (robot description, xacro)
@@ -3,54 +3,97 @@
     <xacro:include filename="$(find maddrive_urdf_tools)/urdf/macros/inertia.urdf.xacro" />
     <xacro:include filename="$(find maddrive_urdf_tools)/urdf/macros/common.urdf.xacro" />
-    <xacro:property name="rs_camera_width" value="0.09" />
-    <xacro:property name="rs_camera_height" value="0.025" />
-    <xacro:property name="rs_camera_length" value="0.025" />
-    <xacro:property name="rs_camera_mass_kg" value="0.320" />
+    <xacro:property name="rs435_camera_mass_kg" value="0.08" />
+    <xacro:property name="rs435_camera_width" value="0.09" />
+    <xacro:property name="rs435_camera_height" value="0.025" />
+    <xacro:property name="rs435_camera_length" value="0.025" />
+    <xacro:property name="rs435_camera_range_min" value="0.4" />
+    <xacro:property name="rs435_camera_range_max" value="4.0" />
+    <xacro:property name="rs455_camera_mass_kg" value="0.11" />
+    <xacro:property name="rs455_camera_width" value="0.124" />
+    <xacro:property name="rs455_camera_height" value="0.029" />
+    <xacro:property name="rs455_camera_length" value="0.026" />
+    <xacro:property name="rs455_camera_range_min" value="0.4" />
+    <xacro:property name="rs455_camera_range_max" value="7.0" />
     <xacro:property name="rs_imu_height" value="0.01" />
     <xacro:property name="rs_imu_width" value="0.01" />
     <xacro:property name="rs_imu_length" value="0.01" />
-    <!-- DEPTH CAMERA -->
     <xacro:macro
-        name="realsense_435"
-        params="name parent xyz rpy">
-        <link name="${name}_link">
+        name="rs_camera"
+        params="prefix model parent origin_xyz origin_rpy">
+        <!-- DEPTH CAMERA -->
+        <joint name="${prefix}_${model}_camera_joint" type="fixed">
+            <parent link="${parent}" />
+            <child link="${prefix}_${model}_camera_link" />
+            <origin xyz="${origin_xyz}" rpy="${origin_rpy}" />
+        </joint>
+        <link name="${prefix}_${model}_camera_link">
             <visual>
+                <origin xyz="0 0 0" rpy="0 0 0" />
                 <geometry>
-                    <box size="${rs_camera_length} ${rs_camera_width} ${rs_camera_height}" />
+                    <xacro:if value="${model == 'rs435'}">
+                        <box size="
+                            ${rs435_camera_length}
+                            ${rs435_camera_width}
+                            ${rs435_camera_height}" />
+                    </xacro:if>
+                    <xacro:if value="${model == 'rs455'}">
+                        <box size="
+                            ${rs455_camera_length}
+                            ${rs455_camera_width}
+                            ${rs455_camera_height}" />
+                    </xacro:if>
                 </geometry>
             </visual>
             <collision>
+                <origin xyz="0 0 0" rpy="0 0 0" />
                 <geometry>
-                    <box size="${rs_camera_length} ${rs_camera_width} ${rs_camera_height}" />
+                    <xacro:if value="${model == 'rs435'}">
+                        <box size="
+                            ${rs435_camera_length}
+                            ${rs435_camera_width}
+                            ${rs435_camera_height}" />
+                    </xacro:if>
+                    <xacro:if value="${model == 'rs455'}">
+                        <box size="
+                            ${rs455_camera_length}
+                            ${rs455_camera_width}
+                            ${rs455_camera_height}" />
+                    </xacro:if>
                 </geometry>
             </collision>
-            <xacro:box_inertia
-                width="${rs_camera_width}"
-                length="${rs_camera_length}"
-                height="${rs_camera_height}"
-                mass="${rs_camera_mass_kg}">
-                <origin xyz="0 0 0" rpy="0 0 0" />
-            </xacro:box_inertia>
+            <xacro:if value="${model == 'rs435'}">
+                <xacro:box_inertia
+                    width="${rs435_camera_width}"
+                    length="${rs435_camera_length}"
+                    height="${rs435_camera_height}"
+                    mass="${rs435_camera_mass_kg}">
+                    <origin xyz="0 0 0" rpy="0 0 0" />
+                </xacro:box_inertia>
+            </xacro:if>
+            <xacro:if value="${model == 'rs455'}">
+                <xacro:box_inertia
+                    width="${rs455_camera_width}"
+                    length="${rs455_camera_length}"
+                    height="${rs455_camera_height}"
+                    mass="${rs455_camera_mass_kg}">
+                    <origin xyz="0 0 0" rpy="0 0 0" />
+                </xacro:box_inertia>
+            </xacro:if>
         </link>
-        <joint name="base_${name}_camera_joint" type="fixed">
-            <parent link="${parent}" />
-            <child link="${name}_link" />
-            <origin xyz="${xyz}" rpy="${rpy}" />
-        </joint>
-        <link name="${name}_optical_frame" />
-        <joint name="${name}_camera_optical_joint" type="fixed">
-            <parent link="${name}_link" />
-            <child link="${name}_optical_frame" />
+        <joint name="${prefix}_${model}_camera_optical_joint" type="fixed">
+            <parent link="${prefix}_${model}_camera_link" />
+            <child link="${prefix}_${model}_camera_optical_frame" />
             <origin xyz="0 0 0" rpy="${-pi/2} 0 ${-pi/2}" />
         </joint>
-        <gazebo reference="${name}_link">
+        <link name="${prefix}_${model}_camera_optical_frame" />
+        <gazebo reference="${prefix}_${model}_camera_link">
             <material>Gazebo/Black</material>
-            <sensor name="${name}" type="depth">
-                <update_rate>20</update_rate>
+            <sensor name="${prefix}_${model}_camera" type="depth">
+                <update_rate>30</update_rate>
                 <camera>
-                    <horizontal_fov>1.29154</horizontal_fov>
+                    <horizontal_fov>1.51844</horizontal_fov>
                     <image>
-                        <width>640</width>
-                        <height>480</height>
+                        <width>1280</width>
+                        <height>720</height>
                         <format>R8G8B8</format>
                     </image>
@@ -60,22 +103,28 @@
                     </clip>
                 </camera>
-                <plugin name="camera_plugin" filename="libgazebo_ros_openni_kinect.so">
+                <plugin name="depth_camera_plugin" filename="libgazebo_ros_openni_kinect.so">
                     <baseline>0.2</baseline>
                     <alwaysOn>true</alwaysOn>
                     <updateRate>20.0</updateRate>
-                    <cameraName>${name}</cameraName>
-                    <imageTopicName>/${name}/color/image_raw</imageTopicName>
-                    <cameraInfoTopicName>/${name}/color/camera_info</cameraInfoTopicName>
-                    <depthImageTopicName>/${name}/aligned_depth_to_color/image_raw</depthImageTopicName>
-                    <depthImageCameraInfoTopicName>/${name}/depth/camera_info</depthImageCameraInfoTopicName>
-                    <pointCloudTopicName>/${name}/depth/color/points</pointCloudTopicName>
-                    <frameName>${name}_optical_frame</frameName>
-                    <pointCloudCutoff>0.05</pointCloudCutoff>
-                    <pointCloudCutoffMax>10</pointCloudCutoffMax>
-                    <distortionK1>0</distortionK1>
-                    <distortionK2>0</distortionK2>
-                    <distortionK3>0</distortionK3>
-                    <distortionT1>0</distortionT1>
-                    <distortionT2>0</distortionT2>
+                    <cameraName>${prefix}_${model}_camera</cameraName>
+                    <imageTopicName>/${prefix}_${model}_camera/color/image_raw</imageTopicName>
+                    <cameraInfoTopicName>/${prefix}_${model}_camera/color/camera_info</cameraInfoTopicName>
+                    <depthImageTopicName>/${prefix}_${model}_camera/aligned_depth_to_color/image_raw</depthImageTopicName>
+                    <depthImageInfoTopicName>/${prefix}_${model}_camera/depth/camera_info</depthImageInfoTopicName>
+                    <pointCloudTopicName>/${prefix}_${model}_camera/depth/color/points</pointCloudTopicName>
+                    <frameName>${prefix}_${model}_camera_optical_frame</frameName>
+                    <xacro:if value="${model == 'rs435'}">
+                        <pointCloudCutoff>${rs435_camera_range_min}</pointCloudCutoff>
+                        <pointCloudCutoffMax>${rs435_camera_range_min}</pointCloudCutoffMax>
+                    </xacro:if>
+                    <xacro:if value="${model == 'rs455'}">
+                        <pointCloudCutoff>${rs455_camera_range_min}</pointCloudCutoff>
+                        <pointCloudCutoffMax>${rs455_camera_range_min}</pointCloudCutoffMax>
+                    </xacro:if>
+                    <distortionK1>0.00000001</distortionK1>
+                    <distortionK2>0.00000001</distortionK2>
+                    <distortionK3>0.00000001</distortionK3>
+                    <distortionT1>0.00000001</distortionT1>
+                    <distortionT2>0.00000001</distortionT2>
                     <CxPrime>0</CxPrime>
                     <Cx>0</Cx>
@@ -87,23 +136,29 @@
         </gazebo>
         <!-- IMU -->
-        <link name="${name}_imu_link">
+        <joint name="${prefix}_${model}_camera_imu_joint" type="fixed">
+            <parent link="${prefix}_${model}_camera_link" />
+            <child link="${prefix}_${model}_camera_imu_link" />
+            <origin xyz="0 0 0" rpy="0 0 0" />
+        </joint>
+        <link name="${prefix}_${model}_camera_imu_link">
             <visual>
                 <geometry>
-                    <box size="${rs_imu_length} ${rs_imu_width} ${rs_imu_height}" />
+                    <box size="
+                        ${rs_imu_length}
+                        ${rs_imu_width}
+                        ${rs_imu_height}" />
                 </geometry>
             </visual>
             <collision>
                 <geometry>
-                    <box size="${rs_imu_length} ${rs_imu_width} ${rs_imu_height}" />
+                    <box size="
+                        ${rs_imu_length}
+                        ${rs_imu_width}
+                        ${rs_imu_height}" />
                 </geometry>
             </collision>
             <xacro:null_inertial />
         </link>
-        <joint name="${name}_camera_imu_joint" type="fixed">
-            <parent link="${name}_link" />
-            <child link="${name}_imu_link" />
-            <origin xyz="0 0 0" rpy="0 0 0" />
-        </joint>
-        <gazebo reference="${name}_imu_link">
+        <gazebo reference="${prefix}_${model}_camera_imu_link">
             <material>Gazebo/Red</material>
             <gravity>true</gravity>
@@ -113,12 +168,12 @@
                 <visualize>true</visualize>
                 <topic>__default_topic__</topic>
-                <plugin filename="libgazebo_ros_imu_sensor.so" name="imu_plugin">
-                    <topicName>/${name}/imu/</topicName>
-                    <bodyName>${name}_imu_link</bodyName>
+                <plugin name="imu_sensor_plugin" filename="libgazebo_ros_imu_sensor.so">
+                    <topicName>/${prefix}_${model}_camera/imu</topicName>
+                    <bodyName>${prefix}_${model}_camera_imu_link</bodyName>
                     <updateRateHZ>20.0</updateRateHZ>
                     <gaussianNoise>0.02</gaussianNoise>
                     <xyzOffset>0 0 0</xyzOffset>
                     <rpyOffset>0 0 0</rpyOffset>
-                    <frameName>${name}_imu_link</frameName>
+                    <frameName>${prefix}_${model}_camera_imu_link</frameName>
                 </plugin>
                 <pose>0 0 0 0 0 0</pose>

File: maddrive_urdf_tools/urdf/macros/sector_lidar.urdf.xacro (robot description, xacro)
@@ -2,5 +2,5 @@
 <robot xmlns:xacro="http://ros.org/wiki/xacro">
     <xacro:include filename="$(find maddrive_urdf_tools)/urdf/macros/inertia.urdf.xacro" />
-    <xacro:property name="c16_lidar_mass" value="1.0" />
+    <xacro:property name="c16_lidar_mass_kg" value="1.0" />
     <xacro:property name="c16_lidar_height" value="0.0779" />
     <xacro:property name="c16_lidar_radius" value="${0.102/2}" />
@@ -13,5 +13,5 @@
     <xacro:property name="c16_lidar_range_min" value="0.5" />
     <xacro:property name="c16_lidar_range_max" value="150" />
-    <xacro:property name="c64_lidar_mass" value="1.0" />
+    <xacro:property name="c64_lidar_mass_kg" value="1.0" />
     <xacro:property name="c64_lidar_height" value="0.09" />
     <xacro:property name="c64_lidar_radius" value="${0.1075/2}" />
@@ -24,21 +24,24 @@
     <xacro:property name="c64_lidar_range_min" value="0.5" />
     <xacro:property name="c64_lidar_range_max" value="100" />
-    <xacro:macro name="sector_lidar" params="model parent origin_xyz origin_rpy">
-        <joint name="${model}_lidar_joint" type="fixed">
-            <axis xyz="0 1 0" />
+    <xacro:macro name="sector_lidar" params="prefix model parent origin_xyz origin_rpy">
+        <joint name="${prefix}_${model}_lidar_joint" type="fixed">
             <parent link="${parent}" />
-            <child link="${model}_lidar_link" />
+            <child link="${prefix}_${model}_lidar_link" />
             <origin xyz="${origin_xyz}" rpy="${origin_rpy}" />
         </joint>
-        <link name="${model}_lidar_link">
+        <link name="${prefix}_${model}_lidar_link">
             <visual>
                 <origin xyz="0 0 0" rpy="0 0 0" />
                 <geometry>
-                <xacro:if value="${model == 'c16'}">
-                    <cylinder length="${c16_lidar_height}" radius="${c16_lidar_radius}" />
-                </xacro:if>
-                <xacro:if value="${model == 'c64'}">
-                    <cylinder length="${c64_lidar_height}" radius="${c64_lidar_radius}" />
-                </xacro:if>
+                    <xacro:if value="${model == 'c16'}">
+                        <cylinder
+                            length="${c16_lidar_height}"
+                            radius="${c16_lidar_radius}" />
+                    </xacro:if>
+                    <xacro:if value="${model == 'c64'}">
+                        <cylinder
+                            length="${c64_lidar_height}"
+                            radius="${c64_lidar_radius}" />
+                    </xacro:if>
                 </geometry>
             </visual>
@@ -46,26 +49,36 @@
                 <origin xyz="0 0 0" rpy="0 0 0" />
                 <geometry>
-                <xacro:if value="${model == 'c16'}">
-                    <cylinder length="${c16_lidar_height}" radius="${c16_lidar_radius}" />
-                </xacro:if>
-                <xacro:if value="${model == 'c64'}">
-                    <cylinder length="${c64_lidar_height}" radius="${c64_lidar_radius}" />
-                </xacro:if>
+                    <xacro:if value="${model == 'c16'}">
+                        <cylinder
+                            length="${c16_lidar_height}"
+                            radius="${c16_lidar_radius}" />
+                    </xacro:if>
+                    <xacro:if value="${model == 'c64'}">
+                        <cylinder
+                            length="${c64_lidar_height}"
+                            radius="${c64_lidar_radius}" />
+                    </xacro:if>
                 </geometry>
             </collision>
             <xacro:if value="${model == 'c16'}">
-                <xacro:cylinder_inertia r="${c16_lidar_radius}" h="${c16_lidar_height}" mass="${c16_lidar_mass}">
+                <xacro:cylinder_inertia
+                    r="${c16_lidar_radius}"
+                    h="${c16_lidar_height}"
+                    mass="${c16_lidar_mass_kg}">
                     <origin xyz="0 0 0" rpy="0 0 0" />
                 </xacro:cylinder_inertia>
             </xacro:if>
             <xacro:if value="${model == 'c64'}">
-                <xacro:cylinder_inertia r="${c64_lidar_radius}" h="${c64_lidar_height}" mass="${c64_lidar_mass}">
+                <xacro:cylinder_inertia
+                    r="${c64_lidar_radius}"
+                    h="${c64_lidar_height}"
+                    mass="${c64_lidar_mass_kg}">
                     <origin xyz="0 0 0" rpy="0 0 0" />
                 </xacro:cylinder_inertia>
             </xacro:if>
         </link>
-        <gazebo reference="${model}_lidar_link">
+        <gazebo reference="${prefix}_${model}_lidar_link">
             <material>Gazebo/Blue</material>
-            <sensor name="${model}_lidar_sensor" type="ray">
+            <sensor name="${prefix}_${model}_lidar_sensor" type="ray">
                 <pose>0 0 0.0 0 0 0</pose>
                 <visualize>true</visualize>
@@ -116,6 +129,6 @@
                 <plugin name="gazebo_ros_block_laser" filename="libgazebo_ros_block_laser.so">
                     <robotNamespace>/</robotNamespace>
-                    <frameName>${model}_lidar_link</frameName>
-                    <topicName>${model}_lidar_points</topicName>
+                    <frameName>${prefix}_${model}_lidar_link</frameName>
+                    <topicName>${prefix}_${model}_lidar_points</topicName>
                     <gaussianNoise>0.01</gaussianNoise>
                     <hokuyoMinIntensity>101</hokuyoMinIntensity>

File: maddrive_urdf_tools/urdf/macros/wheels.urdf.xacro (robot description, xacro)
@@ -1,5 +1,4 @@
 <?xml version="1.0"?>
 <robot xmlns:xacro="http://www.ros.org/wiki/xacro">
-	<xacro:property name="wheel_effort" value="1000000" />
 	<xacro:include filename="$(find maddrive_urdf_tools)/urdf/macros/inertia.urdf.xacro" />
 	<xacro:include filename="$(find maddrive_urdf_tools)/urdf/macros/common.urdf.xacro" />
@@ -26,6 +25,6 @@
 			<material>Gazebo/Black</material>
 			<selfCollide>false</selfCollide>
-            <mu1 value="1.0" />
-            <mu2 value="1.0" />
+			<mu1 value="1.0" />
+			<mu2 value="1.0" />
 		</gazebo>
 	</xacro:macro>
@@ -37,5 +36,5 @@
 			<origin xyz="${origin_xyz}" rpy="0 0 0" />
 			<axis xyz="0 1 0" />
-			<limit effort="${wheel_effort}" velocity="0" />
+			<limit effort="0" velocity="0" />
 		</joint>
 		<xacro:base_wheel name="${prefix}_wheel_link" />
@@ -48,5 +47,5 @@
 			<origin xyz="${steer_origin_xyz}" rpy="0 0 0" />
 			<axis xyz="0 0 1" />
-			<limit lower="${-steer_limit}" upper="${steer_limit}" effort="${wheel_effort}" velocity="0" />
+			<limit lower="${-steer_limit}" upper="${steer_limit}" effort="0" velocity="0" />
 		</joint>
 		<link name="${prefix}_steer_link">
@@ -58,5 +57,5 @@
 			<origin xyz="0 0 0" rpy="0 0 0" />
 			<axis xyz="0 1 0" />
-			<limit effort="${wheel_effort}" velocity="0" />
+			<limit effort="0" velocity="0" />
 		</joint>
 		<xacro:base_wheel name="${prefix}_wheel_link" />
