Commit message: now the camera model is specified explicitly

File: maddrive_urdf_tools/urdf/macros/realsense.urdf.xacro (robot description, xacro)
@@ -3,16 +3,16 @@
     <xacro:include filename="$(find maddrive_urdf_tools)/urdf/macros/inertia.urdf.xacro" />
     <xacro:include filename="$(find maddrive_urdf_tools)/urdf/macros/common.urdf.xacro" />
-    <xacro:property name="rs435_camera_mass_kg" value="0.08" />
-    <xacro:property name="rs435_camera_width" value="0.09" />
-    <xacro:property name="rs435_camera_height" value="0.025" />
-    <xacro:property name="rs435_camera_length" value="0.025" />
-    <xacro:property name="rs435_camera_range_min" value="0.4" />
-    <xacro:property name="rs435_camera_range_max" value="4.0" />
-    <xacro:property name="rs455_camera_mass_kg" value="0.11" />
-    <xacro:property name="rs455_camera_width" value="0.124" />
-    <xacro:property name="rs455_camera_height" value="0.029" />
-    <xacro:property name="rs455_camera_length" value="0.026" />
-    <xacro:property name="rs455_camera_range_min" value="0.4" />
-    <xacro:property name="rs455_camera_range_max" value="7.0" />
+    <xacro:property name="rs_d435i_camera_mass_kg" value="0.08" />
+    <xacro:property name="rs_d435i_camera_width" value="0.09" />
+    <xacro:property name="rs_d435i_camera_height" value="0.025" />
+    <xacro:property name="rs_d435i_camera_length" value="0.025" />
+    <xacro:property name="rs_d435i_camera_range_min" value="0.4" />
+    <xacro:property name="rs_d435i_camera_range_max" value="4.0" />
+    <xacro:property name="rs_d455_camera_mass_kg" value="0.11" />
+    <xacro:property name="rs_d455_camera_width" value="0.124" />
+    <xacro:property name="rs_d455_camera_height" value="0.029" />
+    <xacro:property name="rs_d455_camera_length" value="0.026" />
+    <xacro:property name="rs_d455_camera_range_min" value="0.4" />
+    <xacro:property name="rs_d455_camera_range_max" value="7.0" />
     <xacro:property name="rs_imu_height" value="0.01" />
     <xacro:property name="rs_imu_width" value="0.01" />
@@ -22,24 +22,24 @@
         params="prefix model parent origin_xyz origin_rpy">
         <!-- DEPTH CAMERA -->
-        <joint name="${prefix}_${model}_camera_joint" type="fixed">
+        <joint name="${prefix}_rs_${model}_camera_joint" type="fixed">
             <parent link="${parent}" />
-            <child link="${prefix}_${model}_camera_link" />
+            <child link="${prefix}_rs_${model}_camera_link" />
             <origin xyz="${origin_xyz}" rpy="${origin_rpy}" />
         </joint>
-        <link name="${prefix}_${model}_camera_link">
+        <link name="${prefix}_rs_${model}_camera_link">
             <visual>
                 <origin xyz="0 0 0" rpy="0 0 0" />
                 <geometry>
-                    <xacro:if value="${model == 'rs435'}">
+                    <xacro:if value="${model == 'd435i'}">
                         <box size="
-                            ${rs435_camera_length}
-                            ${rs435_camera_width}
-                            ${rs435_camera_height}" />
+                            ${rs_d435i_camera_length}
+                            ${rs_d435i_camera_width}
+                            ${rs_d435i_camera_height}" />
                     </xacro:if>
-                    <xacro:if value="${model == 'rs455'}">
+                    <xacro:if value="${model == 'd455'}">
                         <box size="
-                            ${rs455_camera_length}
-                            ${rs455_camera_width}
-                            ${rs455_camera_height}" />
+                            ${rs_d455_camera_length}
+                            ${rs_d455_camera_width}
+                            ${rs_d455_camera_height}" />
                     </xacro:if>
                 </geometry>
@@ -48,46 +48,46 @@
                 <origin xyz="0 0 0" rpy="0 0 0" />
                 <geometry>
-                    <xacro:if value="${model == 'rs435'}">
+                    <xacro:if value="${model == 'd435i'}">
                         <box size="
-                            ${rs435_camera_length}
-                            ${rs435_camera_width}
-                            ${rs435_camera_height}" />
+                            ${rs_d435i_camera_length}
+                            ${rs_d435i_camera_width}
+                            ${rs_d435i_camera_height}" />
                     </xacro:if>
-                    <xacro:if value="${model == 'rs455'}">
+                    <xacro:if value="${model == 'd455'}">
                         <box size="
-                            ${rs455_camera_length}
-                            ${rs455_camera_width}
-                            ${rs455_camera_height}" />
+                            ${rs_d455_camera_length}
+                            ${rs_d455_camera_width}
+                            ${rs_d455_camera_height}" />
                     </xacro:if>
                 </geometry>
             </collision>
-            <xacro:if value="${model == 'rs435'}">
+            <xacro:if value="${model == 'd435i'}">
                 <xacro:box_inertia
-                    width="${rs435_camera_width}"
-                    length="${rs435_camera_length}"
-                    height="${rs435_camera_height}"
-                    mass="${rs435_camera_mass_kg}">
+                    width="${rs_d435i_camera_width}"
+                    length="${rs_d435i_camera_length}"
+                    height="${rs_d435i_camera_height}"
+                    mass="${rs_d435i_camera_mass_kg}">
                     <origin xyz="0 0 0" rpy="0 0 0" />
                 </xacro:box_inertia>
             </xacro:if>
-            <xacro:if value="${model == 'rs455'}">
+            <xacro:if value="${model == 'd455'}">
                 <xacro:box_inertia
-                    width="${rs455_camera_width}"
-                    length="${rs455_camera_length}"
-                    height="${rs455_camera_height}"
-                    mass="${rs455_camera_mass_kg}">
+                    width="${rs_d455_camera_width}"
+                    length="${rs_d455_camera_length}"
+                    height="${rs_d455_camera_height}"
+                    mass="${rs_d455_camera_mass_kg}">
                     <origin xyz="0 0 0" rpy="0 0 0" />
                 </xacro:box_inertia>
             </xacro:if>
         </link>
-        <joint name="${prefix}_${model}_camera_optical_joint" type="fixed">
-            <parent link="${prefix}_${model}_camera_link" />
-            <child link="${prefix}_${model}_camera_optical_frame" />
+        <joint name="${prefix}_rs_${model}_camera_optical_joint" type="fixed">
+            <parent link="${prefix}_rs_${model}_camera_link" />
+            <child link="${prefix}_rs_${model}_camera_optical_frame" />
             <origin xyz="0 0 0" rpy="${-pi/2} 0 ${-pi/2}" />
         </joint>
-        <link name="${prefix}_${model}_camera_optical_frame" />
-        <gazebo reference="${prefix}_${model}_camera_link">
+        <link name="${prefix}_rs_${model}_camera_optical_frame" />
+        <gazebo reference="${prefix}_rs_${model}_camera_link">
             <material>Gazebo/Black</material>
-            <sensor name="${prefix}_${model}_camera" type="depth">
+            <sensor name="${prefix}_rs_${model}_camera" type="depth">
                 <update_rate>30</update_rate>
                 <camera>
@@ -107,18 +107,18 @@
                     <alwaysOn>true</alwaysOn>
                     <updateRate>20.0</updateRate>
-                    <cameraName>${prefix}_${model}_camera</cameraName>
-                    <imageTopicName>/${prefix}_${model}_camera/color/image_raw</imageTopicName>
-                    <cameraInfoTopicName>/${prefix}_${model}_camera/color/camera_info</cameraInfoTopicName>
-                    <depthImageTopicName>/${prefix}_${model}_camera/aligned_depth_to_color/image_raw</depthImageTopicName>
-                    <depthImageInfoTopicName>/${prefix}_${model}_camera/depth/camera_info</depthImageInfoTopicName>
-                    <pointCloudTopicName>/${prefix}_${model}_camera/depth/color/points</pointCloudTopicName>
-                    <frameName>${prefix}_${model}_camera_optical_frame</frameName>
-                    <xacro:if value="${model == 'rs435'}">
-                        <pointCloudCutoff>${rs435_camera_range_min}</pointCloudCutoff>
-                        <pointCloudCutoffMax>${rs435_camera_range_min}</pointCloudCutoffMax>
+                    <cameraName>${prefix}_rs_${model}_camera</cameraName>
+                    <imageTopicName>/${prefix}_rs_${model}_camera/color/image_raw</imageTopicName>
+                    <cameraInfoTopicName>/${prefix}_rs_${model}_camera/color/camera_info</cameraInfoTopicName>
+                    <depthImageTopicName>/${prefix}_rs_${model}_camera/aligned_depth_to_color/image_raw</depthImageTopicName>
+                    <depthImageInfoTopicName>/${prefix}_rs_${model}_camera/depth/camera_info</depthImageInfoTopicName>
+                    <pointCloudTopicName>/${prefix}_rs_${model}_camera/depth/color/points</pointCloudTopicName>
+                    <frameName>${prefix}_rs_${model}_camera_optical_frame</frameName>
+                    <xacro:if value="${model == 'rs_d435i'}">
+                        <pointCloudCutoff>${rs_d435i_camera_range_min}</pointCloudCutoff>
+                        <pointCloudCutoffMax>${rs_d435i_camera_range_min}</pointCloudCutoffMax>
                     </xacro:if>
-                    <xacro:if value="${model == 'rs455'}">
-                        <pointCloudCutoff>${rs455_camera_range_min}</pointCloudCutoff>
-                        <pointCloudCutoffMax>${rs455_camera_range_min}</pointCloudCutoffMax>
+                    <xacro:if value="${model == 'rs_d455'}">
+                        <pointCloudCutoff>${rs_d455_camera_range_min}</pointCloudCutoff>
+                        <pointCloudCutoffMax>${rs_d455_camera_range_min}</pointCloudCutoffMax>
                     </xacro:if>
                     <distortionK1>0.00000001</distortionK1>
@@ -136,10 +136,10 @@
         </gazebo>
         <!-- IMU -->
-        <joint name="${prefix}_${model}_camera_imu_joint" type="fixed">
-            <parent link="${prefix}_${model}_camera_link" />
-            <child link="${prefix}_${model}_camera_imu_link" />
+        <joint name="${prefix}_rs_${model}_camera_imu_joint" type="fixed">
+            <parent link="${prefix}_rs_${model}_camera_link" />
+            <child link="${prefix}_rs_${model}_camera_imu_link" />
             <origin xyz="0 0 0" rpy="0 0 0" />
         </joint>
-        <link name="${prefix}_${model}_camera_imu_link">
+        <link name="${prefix}_rs_${model}_camera_imu_link">
             <visual>
                 <geometry>
@@ -160,5 +160,5 @@
             <xacro:null_inertial />
         </link>
-        <gazebo reference="${prefix}_${model}_camera_imu_link">
+        <gazebo reference="${prefix}_rs_${model}_camera_imu_link">
             <material>Gazebo/Red</material>
             <gravity>true</gravity>
@@ -169,11 +169,11 @@
                 <topic>__default_topic__</topic>
                 <plugin name="imu_sensor_plugin" filename="libgazebo_ros_imu_sensor.so">
-                    <topicName>/${prefix}_${model}_camera/imu</topicName>
-                    <bodyName>${prefix}_${model}_camera_imu_link</bodyName>
+                    <topicName>/${prefix}_rs_${model}_camera/imu</topicName>
+                    <bodyName>${prefix}_rs_${model}_camera_imu_link</bodyName>
                     <updateRateHZ>20.0</updateRateHZ>
                     <gaussianNoise>0.02</gaussianNoise>
                     <xyzOffset>0 0 0</xyzOffset>
                     <rpyOffset>0 0 0</rpyOffset>
-                    <frameName>${prefix}_${model}_camera_imu_link</frameName>
+                    <frameName>${prefix}_rs_${model}_camera_imu_link</frameName>
                 </plugin>
                 <pose>0 0 0 0 0 0</pose>

Commit message: changed the orientation of the coordinate system of the IMU sensor according to the description

File: maddrive_urdf_tools/urdf/macros/realsense.urdf.xacro (robot description, xacro)
@@ -139,5 +139,5 @@
             <parent link="${prefix}_rs_${model}_camera_link" />
             <child link="${prefix}_rs_${model}_camera_imu_link" />
-            <origin xyz="0 0 0" rpy="0 0 0" />
+            <origin xyz="0 0 0" rpy="${-pi/2} 0 ${-pi/2}" /> <!-- realsense2_description/launch/view_d435i(d455)_model.launch -->
         </joint>
         <link name="${prefix}_rs_${model}_camera_imu_link">
