Commit message: modified the lidar macro as common as all macros

File: maddrive_urdf_tools/urdf/macros/lidar.urdf.xacro (robot description, xacro)
@@ -4,12 +4,17 @@
     <xacro:property name="lidar_height" value="0.02" />
     <xacro:property name="lidar_radius" value="0.04" />
-    <xacro:macro name="simple_lidar" params="name parent place_height">
-        <link name="${name}">
-            <cylinder_inertial
-                radius="${lidar_radius}"
-                length="${lidar_height}"
-                mass="${lidar_mass}">
+    <xacro:macro name="lidar" params="prefix parent origin_xyz origin_rpy">
+        <joint name="${prefix}_lidar_joint" type="fixed">
+            <parent link="${parent}" />
+            <child link="${prefix}_lidar_link" />
+            <origin xyz="${origin_xyz}" rpy="${origin_rpy}" />
+        </joint>
+        <link name="${prefix}_lidar_link">
+            <visual>
                 <origin xyz="0 0 0" rpy="0 0 0" />
-            </cylinder_inertial>
+                <geometry>
+                    <cylinder length="${lidar_height}" radius="${lidar_radius}" />
+                </geometry>
+            </visual>
             <collision>
                 <origin xyz="0 0 0" rpy="0 0 0" />
@@ -18,29 +23,25 @@
                 </geometry>
             </collision>
-            <visual>
+            <xacro:cylinder_inertia
+                radius="${lidar_radius}"
+                length="${lidar_height}"
+                mass="${lidar_mass}">
                 <origin xyz="0 0 0" rpy="0 0 0" />
-                <geometry>
-                    <cylinder length="${lidar_height}" radius="${lidar_radius}" />
-                </geometry>
-            </visual>
+            </xacro:cylinder_inertia>
         </link>
-        <joint name="lidar_joint" type="fixed">
-            <parent link="${parent}" />
-            <child link="lidar_link" />
-            <origin xyz="0 0 ${place_height}" rpy="0 0 0" />
-        </joint>
-        <gazebo reference="lidar_link">
+        <gazebo reference="${prefix}_lidar_link">
+            <selfCollide>false</selfCollide>
             <material>Gazebo/Red</material>
-            <sensor name="head_hokuyo_sensor" type="ray">
+            <sensor name="${prefix}_lidar_sensor" type="ray">
                 <pose>0 0 0 0 0 0</pose>
-                <visualize>false</visualize>
-                <update_rate>40</update_rate>
+                <visualize>true</visualize>
+                <update_rate>10</update_rate>
                 <ray>
                     <scan>
                         <horizontal>
-                            <samples>720</samples>
+                            <samples>360</samples>
                             <resolution>1</resolution>
-                            <min_angle>-3.14</min_angle>
-                            <max_angle>3.14</max_angle>
+                            <min_angle>${-pi}</min_angle>
+                            <max_angle>${pi}</max_angle>
                         </horizontal>
                     </scan>
@@ -53,10 +54,10 @@
                         <type>gaussian</type>
                         <mean>0.0</mean>
-                        <stddev>0.01</stddev>
+                        <stddev>0.03</stddev>
                     </noise>
                 </ray>
-                <plugin name="gazebo_ros_head_hokuyo_controller" filename="libgazebo_ros_laser.so">
-                    <topicName>/scan</topicName>
-                    <frameName>lidar_link</frameName>
+                <plugin name="gazebo_ros_lidar_controller" filename="libgazebo_ros_laser.so">
+                    <topicName>${prefix}_lidar_scan</topicName>
+                    <frameName>${prefix}_lidar_link</frameName>
                 </plugin>
             </sensor>

Commit message: add real ydlidar sizes (TODO scan offset in urdf (43 mm))

File: maddrive_urdf_tools/urdf/macros/lidar.urdf.xacro (robot description, xacro)
@@ -2,6 +2,6 @@
 <robot xmlns:xacro="http://www.ros.org/wiki/xacro">
     <xacro:property name="lidar_mass" value="0.1" />
-    <xacro:property name="lidar_height" value="0.02" />
-    <xacro:property name="lidar_radius" value="0.04" />
+    <xacro:property name="lidar_height" value="0.016" />
+    <xacro:property name="lidar_radius" value="0.03" />
     <xacro:macro name="lidar" params="prefix parent origin_xyz origin_rpy">
         <joint name="${prefix}_lidar_joint" type="fixed">

Commit message: add lidar base and suspention parameters in urdf macros

File: maddrive_urdf_tools/urdf/macros/lidar.urdf.xacro (robot description, xacro)
@@ -4,11 +4,22 @@
     <xacro:property name="lidar_height" value="0.016" />
     <xacro:property name="lidar_radius" value="0.03" />
+    <xacro:property name="lidar_base_2_scan_offset_z" value="0.043" />
     <xacro:macro name="lidar" params="prefix parent origin_xyz origin_rpy">
-        <joint name="${prefix}_lidar_joint" type="fixed">
+        <joint name="${prefix}_lidar_base_joint" type="fixed">
             <parent link="${parent}" />
-            <child link="${prefix}_lidar_link" />
+            <child link="${prefix}_lidar_base_link" />
             <origin xyz="${origin_xyz}" rpy="${origin_rpy}" />
         </joint>
-        <link name="${prefix}_lidar_link">
+        <link name="${prefix}_lidar_base_link">
+            <xacro:null_visual/>
+            <xacro:null_collision/>
+            <xacro:null_inertia/>
+        </link>
+        <joint name="${prefix}_lidar_scan_joint" type="fixed">
+            <parent link="${prefix}_lidar_base_link" />
+            <child link="${prefix}_lidar_scan_link" />
+            <origin xyz="0 0 ${lidar_base_2_scan_offset_z}" rpy="0 0 0" />
+        </joint>
+        <link name="${prefix}_lidar_scan_link">
             <visual>
                 <origin xyz="0 0 0" rpy="0 0 0" />
@@ -30,8 +41,8 @@
             </xacro:cylinder_inertia>
         </link>
-        <gazebo reference="${prefix}_lidar_link">
+        <gazebo reference="${prefix}_lidar_scan_link">
             <selfCollide>false</selfCollide>
             <material>Gazebo/Red</material>
-            <sensor name="${prefix}_lidar_sensor" type="ray">
+            <sensor name="${prefix}_lidar_scan_sensor" type="ray">
                 <pose>0 0 0 0 0 0</pose>
                 <visualize>true</visualize>
@@ -59,5 +70,5 @@
                 <plugin name="gazebo_ros_lidar_controller" filename="libgazebo_ros_laser.so">
                     <topicName>${prefix}_lidar_scan/raw</topicName>
-                    <frameName>${prefix}_lidar_link</frameName>
+                    <frameName>${prefix}_lidar_scan_link</frameName>
                 </plugin>
             </sensor>

File: maddrive_urdf_tools/urdf/macros/wheels.urdf.xacro (robot description, xacro)
@@ -34,9 +34,19 @@
 	</xacro:macro>
 	<!-- SPEED WHEEL -->
-	<xacro:macro name="speed_wheel" params="prefix parent origin_xyz ">
+	<xacro:macro name="speed_wheel" params="prefix parent suspension_origin_xyz ">
+		<joint name="${prefix}_suspension_joint" type="fixed">
+			<parent link="${parent}" />
+			<child link="${prefix}_suspension_link" />
+			<origin xyz="${suspension_origin_xyz}" rpy="0 0 0" />
+		</joint>
+		<link name="${prefix}_suspension_link">
+			<xacro:null_visual/>
+			<xacro:null_collision/>
+			<xacro:null_inertia/>
+		</link>
 		<joint name="${prefix}_wheel_joint" type="continuous">
-			<parent link="${parent}" />
+			<parent link="${prefix}_suspension_link" />
 			<child link="${prefix}_wheel_link" />
-			<origin xyz="${origin_xyz}" rpy="0 0 0" />
+			<origin xyz="0 0 -${suspension_height}" rpy="0 0 0" />
 			<axis xyz="0 1 0" />
 			<limit effort="100000" velocity="${pi*10}" />
@@ -55,9 +65,19 @@
 	</xacro:macro>
 	<!-- STEER WHEEL -->
-	<xacro:macro name="steer_wheel" params="prefix parent steer_origin_xyz steer_limit">
+	<xacro:macro name="steer_wheel" params="prefix parent suspension_origin_xyz suspension_height steer_limit">
+		<joint name="${prefix}_suspension_joint" type="fixed">
+			<parent link="${parent}" />
+			<child link="${prefix}_suspension_link" />
+			<origin xyz="${suspension_origin_xyz}" rpy="0 0 0" />
+		</joint>
+		<link name="${prefix}_suspension_link">
+			<xacro:null_visual/>
+			<xacro:null_collision/>
+			<xacro:null_inertia/>
+		</link>
 		<joint name="${prefix}_steer_joint" type="revolute">
-			<parent link="${parent}" />
+			<parent link="${prefix}_suspension_link" />
 			<child link="${prefix}_steer_link" />
-			<origin xyz="${steer_origin_xyz}" rpy="0 0 0" />
+			<origin xyz="0 0 -${suspension_height}" rpy="0 0 0" />
 			<axis xyz="0 0 1" />
 			<limit lower="${-steer_limit}" upper="${steer_limit}" effort="100000" velocity="${pi*2}" />
