Commit message: ydlidar macros

File: maddrive_urdf_tools/urdf/macros/ydlidar.urdf.xacro (robot description, xacro)
@@ -1,29 +1,29 @@
 <?xml version="1.0"?>
 <robot xmlns:xacro="http://www.ros.org/wiki/xacro">
-    <xacro:property name="lidar_mass" value="0.1" />
-    <xacro:property name="lidar_height" value="0.016" />
-    <xacro:property name="lidar_radius" value="0.03" />
-    <xacro:property name="lidar_base_2_scan_offset_z" value="0.043" />
-    <xacro:macro name="lidar" params="prefix parent origin_xyz origin_rpy">
-        <joint name="${prefix}_lidar_base_joint" type="fixed">
+    <xacro:property name="ydlidar_mass" value="0.1" />
+    <xacro:property name="ydlidar_height" value="0.016" />
+    <xacro:property name="ydlidar_radius" value="0.03" />
+    <xacro:property name="ydlidar_base_2_scan_offset_z" value="0.043" />
+    <xacro:macro name="ydlidar" params="prefix parent origin_xyz origin_rpy">
+        <joint name="${prefix}_ydlidar_base_joint" type="fixed">
             <parent link="${parent}" />
-            <child link="${prefix}_lidar_base_link" />
+            <child link="${prefix}_ydlidar_base_link" />
             <origin xyz="${origin_xyz}" rpy="${origin_rpy}" />
         </joint>
-        <link name="${prefix}_lidar_base_link">
+        <link name="${prefix}_ydlidar_base_link">
             <xacro:null_visual/>
             <xacro:null_collision/>
             <xacro:null_inertia/>
         </link>
-        <joint name="${prefix}_lidar_scan_joint" type="fixed">
-            <parent link="${prefix}_lidar_base_link" />
-            <child link="${prefix}_lidar_scan_link" />
-            <origin xyz="0 0 ${lidar_base_2_scan_offset_z}" rpy="0 0 0" />
+        <joint name="${prefix}_ydlidar_scan_joint" type="fixed">
+            <parent link="${prefix}_ydlidar_base_link" />
+            <child link="${prefix}_ydlidar_scan_link" />
+            <origin xyz="0 0 ${ydlidar_base_2_scan_offset_z}" rpy="0 0 0" />
         </joint>
-        <link name="${prefix}_lidar_scan_link">
+        <link name="${prefix}_ydlidar_scan_link">
             <visual>
                 <origin xyz="0 0 0" rpy="0 0 0" />
                 <geometry>
-                    <cylinder length="${lidar_height}" radius="${lidar_radius}" />
+                    <cylinder length="${ydlidar_height}" radius="${ydlidar_radius}" />
                 </geometry>
             </visual>
@@ -31,18 +31,18 @@
                 <origin xyz="0 0 0" rpy="0 0 0" />
                 <geometry>
-                    <cylinder length="${lidar_height}" radius="${lidar_radius}" />
+                    <cylinder length="${ydlidar_height}" radius="${ydlidar_radius}" />
                 </geometry>
             </collision>
             <xacro:cylinder_inertia
-                radius="${lidar_radius}"
-                length="${lidar_height}"
-                mass="${lidar_mass}">
+                radius="${ydlidar_radius}"
+                length="${ydlidar_height}"
+                mass="${ydlidar_mass}">
                 <origin xyz="0 0 0" rpy="0 0 0" />
             </xacro:cylinder_inertia>
         </link>
-        <gazebo reference="${prefix}_lidar_scan_link">
+        <gazebo reference="${prefix}_ydlidar_scan_link">
             <selfCollide>false</selfCollide>
             <material>Gazebo/Red</material>
-            <sensor name="${prefix}_lidar_scan_sensor" type="ray">
+            <sensor name="${prefix}_ydlidar_scan_sensor" type="ray">
                 <pose>0 0 0 0 0 0</pose>
                 <visualize>true</visualize>
@@ -68,7 +68,7 @@
                     </noise>
                 </ray>
-                <plugin name="gazebo_ros_lidar_controller" filename="libgazebo_ros_laser.so">
-                    <topicName>${prefix}_lidar_scan/raw</topicName>
-                    <frameName>${prefix}_lidar_scan_link</frameName>
+                <plugin name="gazebo_ros_laser" filename="libgazebo_ros_laser.so">
+                    <topicName>${prefix}_ydlidar_scan/raw</topicName>
+                    <frameName>${prefix}_ydlidar_scan_link</frameName>
                 </plugin>
             </sensor>

Commit message: removed ydlidar base (useless)

File: maddrive_urdf_tools/urdf/macros/ydlidar.urdf.xacro (robot description, xacro)
@@ -4,20 +4,9 @@
     <xacro:property name="ydlidar_height" value="0.016" />
     <xacro:property name="ydlidar_radius" value="0.03" />
-    <xacro:property name="ydlidar_base_2_scan_offset_z" value="0.043" />
     <xacro:macro name="ydlidar" params="prefix parent origin_xyz origin_rpy">
-        <joint name="${prefix}_ydlidar_base_joint" type="fixed">
+        <joint name="${prefix}_ydlidar_scan_joint" type="fixed">
             <parent link="${parent}" />
-            <child link="${prefix}_ydlidar_base_link" />
+            <child link="${prefix}_ydlidar_scan_link" />
             <origin xyz="${origin_xyz}" rpy="${origin_rpy}" />
-        </joint>
-        <link name="${prefix}_ydlidar_base_link">
-            <xacro:null_visual/>
-            <xacro:null_collision/>
-            <xacro:null_inertia/>
-        </link>
-        <joint name="${prefix}_ydlidar_scan_joint" type="fixed">
-            <parent link="${prefix}_ydlidar_base_link" />
-            <child link="${prefix}_ydlidar_scan_link" />
-            <origin xyz="0 0 ${ydlidar_base_2_scan_offset_z}" rpy="0 0 0" />
         </joint>
         <link name="${prefix}_ydlidar_scan_link">
@@ -44,5 +33,5 @@
             <selfCollide>false</selfCollide>
             <material>Gazebo/Red</material>
-            <sensor name="${prefix}_ydlidar_scan_sensor" type="ray">
+            <sensor name="${prefix}_ydlidar_sensor" type="ray">
                 <pose>0 0 0 0 0 0</pose>
                 <visualize>true</visualize>
