Commit message: unsuccessful tries to configure the gps plugin

File: maddrive_urdf_tools/urdf/macros/gps.urdf.xacro (robot description, xacro)
@@ -33,23 +33,30 @@
             </xacro:box_inertia>
         </link>
-    <gazebo reference="gps_link">
-        <material>Gazebo/Orange</material>
-        <plugin name="gazebo_ros_gps" filename="libhector_gazebo_ros_gps.so">
-            <updateRate>4.0</updateRate>
-            <bodyName>gps_link</bodyName>
-            <frameId>gps_link</frameId>
-            <topicName>/gps/fix</topicName>
-            <velocityTopicName>/gps/fix_velocity</velocityTopicName>
-            <referenceLatitude>-30.06022459407145675</referenceLatitude>
-            <referenceLongitude>-51.173913575780311191</referenceLongitude>
-            <referenceHeading>90</referenceHeading>
-            <referenceAltitude>10</referenceAltitude>
-            <offset>0 0 0</offset>
-            <drift>0.001 0.001 0.001</drift>
-            <gaussianNoise>0.05 0.05 0.05</gaussianNoise>
-            <velocityDrift>0.001 0.001 0.001</velocityDrift>
-            <velocityGaussianNoise>0.5 0.5 0.5</velocityGaussianNoise>
-        </plugin>
-    </gazebo>
+        <!-- http://wiki.ros.org/hector_gazebo_plugins -->
+        <gazebo reference="gps_link">
+            <material>Gazebo/Orange</material>
+            <plugin name="gazebo_ros_gps" filename="libhector_gazebo_ros_gps.so">
+                <updateRate>4.0</updateRate>
+                <!-- <robotNamespace>/</robotNamespace> -->
+                <bodyName>gps_link</bodyName>
+                <frameId>/world</frameId>
+                <topicName>/gps/fix</topicName>
+                <velocityTopicName>/gps/vel</velocityTopicName>
+                <referenceLatitude>-30.06022459407145675</referenceLatitude>
+                <referenceLongitude>-51.173913575780311191</referenceLongitude>
+                <referenceHeading>90</referenceHeading>
+                <referenceAltitude>10</referenceAltitude>
+                <!-- <status>10</status> -->
+                <!-- <service>10</service> -->
+                <offset>0.0 0.0 0.0</offset>
+                <drift>0.001 0.001 0.001</drift>
+                <driftFrequency>0.001 0.001 0.001</driftFrequency>
+                <gaussianNoise>0.05 0.05 0.05</gaussianNoise>
+                <velocityOffset>0.001 0.001 0.001</velocityOffset>
+                <velocityDrift>0.001 0.001 0.001</velocityDrift>
+                <velocityDriftFrequency>0.001 0.001 0.001</velocityDriftFrequency>
+                <velocityGaussianNoise>0.5 0.5 0.5</velocityGaussianNoise>
+            </plugin>
+        </gazebo>
     </xacro:macro>
 </robot>

Commit message: added a package with additional plugins for gazebo; renamed the topics created by the sector lidar plugin; solved the problem with the gps plugin

File: maddrive_urdf_tools/urdf/macros/gps.urdf.xacro (robot description, xacro)
@@ -2,19 +2,19 @@
 <robot xmlns:xacro="http://ros.org/wiki/xacro">
     <xacro:include filename="$(find maddrive_urdf_tools)/urdf/macros/inertia.urdf.xacro" />
-    <xacro:property name="gps_length" value="0.05" />
-    <xacro:property name="gps_width" value="0.05" />
-    <xacro:property name="gps_height" value="0.05" />
-    <xacro:property name="gps_mass" value="0.1" />
-    <xacro:macro name="gps" params="parent origin_xyz origin_rpy">
-        <joint name="gps_joint" type="fixed">
+    <xacro:property name="gps_sensor_length" value="0.05" />
+    <xacro:property name="gps_sensor_width" value="0.05" />
+    <xacro:property name="gps_sensor_height" value="0.05" />
+    <xacro:property name="gps_sensor_mass" value="0.1" />
+    <xacro:macro name="gps_sensor" params="prefix parent origin_xyz origin_rpy">
+        <joint name="${prefix}_gps_sensor_joint" type="fixed">
             <parent link="${parent}" />
-            <child link="gps_link" />
+            <child link="${prefix}_gps_sensor_link" />
             <origin xyz="${origin_xyz}" rpy="${origin_rpy}" />
         </joint>
-        <link name="gps_link">
+        <link name="${prefix}_gps_sensor_link">
             <collision>
                 <origin xyz="0 0 0" rpy="0 0 0" />
                 <geometry>
-                    <box size="${gps_length} ${gps_width} ${gps_height}" />
+                    <box size="${gps_sensor_length} ${gps_sensor_width} ${gps_sensor_height}" />
                 </geometry>
             </collision>
@@ -22,29 +22,28 @@
                 <origin xyz="0 0 0" rpy="0 0 0" />
                 <geometry>
-                    <box size="${gps_length} ${gps_width} ${gps_height}" />
+                    <box size="${gps_sensor_length} ${gps_sensor_width} ${gps_sensor_height}" />
                 </geometry>
             </visual>
             <xacro:box_inertia
-                length="${gps_length}"
-                width="${gps_width}"
-                height="${gps_height}"
-                mass="${gps_mass}">
+                length="${gps_sensor_length}"
+                width="${gps_sensor_width}"
+                height="${gps_sensor_height}"
+                mass="${gps_sensor_mass}">
                 <origin xyz="0 0 0" rpy="0 0 0" />
             </xacro:box_inertia>
         </link>
         <!-- http://wiki.ros.org/hector_gazebo_plugins -->
-        <gazebo reference="gps_link">
-            <material>Gazebo/Orange</material>
-            <plugin name="gazebo_ros_gps" filename="libhector_gazebo_ros_gps.so">
+        <gazebo>
+            <plugin name="gazebo_ros_gps_sensor" filename="libhector_gazebo_ros_gps.so">
                 <updateRate>4.0</updateRate>
                 <!-- <robotNamespace>/</robotNamespace> -->
-                <bodyName>gps_link</bodyName>
-                <frameId>/world</frameId>
-                <topicName>/gps/fix</topicName>
-                <velocityTopicName>/gps/vel</velocityTopicName>
+                <bodyName>${prefix}_gps_sensor_link</bodyName>
+                <frameId>${prefix}_gps_sensor</frameId>
+                <topicName>${prefix}_gps_sensor/fix</topicName>
+                <velocityTopicName>${prefix}_gps_sensor/vel</velocityTopicName>
                 <referenceLatitude>-30.06022459407145675</referenceLatitude>
                 <referenceLongitude>-51.173913575780311191</referenceLongitude>
-                <referenceHeading>90</referenceHeading>
-                <referenceAltitude>10</referenceAltitude>
+                <referenceHeading>90.0</referenceHeading>
+                <referenceAltitude>10.0</referenceAltitude>
                 <!-- <status>10</status> -->
                 <!-- <service>10</service> -->

File: maddrive_urdf_tools/urdf/macros/sector_lidar.urdf.xacro (robot description, xacro)
@@ -2,33 +2,33 @@
 <robot xmlns:xacro="http://ros.org/wiki/xacro">
     <xacro:include filename="$(find maddrive_urdf_tools)/urdf/macros/inertia.urdf.xacro" />
-    <xacro:property name="c16_lidar_mass_kg" value="1.0" />
-    <xacro:property name="c16_lidar_height" value="0.0779" />
-    <xacro:property name="c16_lidar_radius" value="${0.102/2}" />
-    <xacro:property name="c16_lidar_hz" value="20" />
-    <xacro:property name="c16_lidar_number_of_channels" value="16" />
-    <xacro:property name="c16_lidar_horizontal_min_angle" value="-${pi}" />
-    <xacro:property name="c16_lidar_horizontal_max_angle" value="${pi}" />
-    <xacro:property name="c16_lidar_vertical_min_angle" value="-0.261799" />
-    <xacro:property name="c16_lidar_vertical_max_angle" value="0.261799" />
-    <xacro:property name="c16_lidar_range_min" value="0.5" />
-    <xacro:property name="c16_lidar_range_max" value="150" />
-    <xacro:property name="c64_lidar_mass_kg" value="1.0" />
-    <xacro:property name="c64_lidar_height" value="0.09" />
-    <xacro:property name="c64_lidar_radius" value="${0.1075/2}" />
-    <xacro:property name="c64_lidar_hz" value="20" />
-    <xacro:property name="c64_lidar_number_of_channels" value="64" />
-    <xacro:property name="c64_lidar_horizontal_min_angle" value="-${pi/2}" />
-    <xacro:property name="c64_lidar_horizontal_max_angle" value="${pi/2}" />
-    <xacro:property name="c64_lidar_vertical_min_angle" value="-0.436332" />
-    <xacro:property name="c64_lidar_vertical_max_angle" value="0.261799" />
-    <xacro:property name="c64_lidar_range_min" value="0.5" />
-    <xacro:property name="c64_lidar_range_max" value="100" />
+    <xacro:property name="c16_mass_kg" value="1.0" />
+    <xacro:property name="c16_height" value="0.0779" />
+    <xacro:property name="c16_radius" value="${0.102/2}" />
+    <xacro:property name="c16_hz" value="20" />
+    <xacro:property name="c16_number_of_channels" value="16" />
+    <xacro:property name="c16_horizontal_min_angle" value="-${pi}" />
+    <xacro:property name="c16_horizontal_max_angle" value="${pi}" />
+    <xacro:property name="c16_vertical_min_angle" value="-0.261799" />
+    <xacro:property name="c16_vertical_max_angle" value="0.261799" />
+    <xacro:property name="c16_range_min" value="0.5" />
+    <xacro:property name="c16_range_max" value="150" />
+    <xacro:property name="c64_mass_kg" value="1.0" />
+    <xacro:property name="c64_height" value="0.09" />
+    <xacro:property name="c64_radius" value="${0.1075/2}" />
+    <xacro:property name="c64_hz" value="20" />
+    <xacro:property name="c64_number_of_channels" value="64" />
+    <xacro:property name="c64_horizontal_min_angle" value="-${pi/2}" />
+    <xacro:property name="c64_horizontal_max_angle" value="${pi/2}" />
+    <xacro:property name="c64_vertical_min_angle" value="-0.436332" />
+    <xacro:property name="c64_vertical_max_angle" value="0.261799" />
+    <xacro:property name="c64_range_min" value="0.5" />
+    <xacro:property name="c64_range_max" value="100" />
     <xacro:macro name="sector_lidar" params="prefix model parent origin_xyz origin_rpy">
-        <joint name="${prefix}_${model}_lidar_joint" type="fixed">
+        <joint name="${prefix}_lslidar_${model}_lidar_joint" type="fixed">
             <parent link="${parent}" />
-            <child link="${prefix}_${model}_lidar_link" />
+            <child link="${prefix}_lslidar_${model}_lidar_link" />
             <origin xyz="${origin_xyz}" rpy="${origin_rpy}" />
         </joint>
-        <link name="${prefix}_${model}_lidar_link">
+        <link name="${prefix}_lslidar_${model}_lidar_link">
             <visual>
                 <origin xyz="0 0 0" rpy="0 0 0" />
@@ -36,11 +36,11 @@
                     <xacro:if value="${model == 'c16'}">
                         <cylinder
-                            length="${c16_lidar_height}"
-                            radius="${c16_lidar_radius}" />
+                            length="${c16_height}"
+                            radius="${c16_radius}" />
                     </xacro:if>
                     <xacro:if value="${model == 'c64'}">
                         <cylinder
-                            length="${c64_lidar_height}"
-                            radius="${c64_lidar_radius}" />
+                            length="${c64_height}"
+                            radius="${c64_radius}" />
                     </xacro:if>
                 </geometry>
@@ -51,11 +51,11 @@
                     <xacro:if value="${model == 'c16'}">
                         <cylinder
-                            length="${c16_lidar_height}"
-                            radius="${c16_lidar_radius}" />
+                            length="${c16_height}"
+                            radius="${c16_radius}" />
                     </xacro:if>
                     <xacro:if value="${model == 'c64'}">
                         <cylinder
-                            length="${c64_lidar_height}"
-                            radius="${c64_lidar_radius}" />
+                            length="${c64_height}"
+                            radius="${c64_radius}" />
                     </xacro:if>
                 </geometry>
@@ -63,7 +63,7 @@
             <xacro:if value="${model == 'c16'}">
                 <xacro:cylinder_inertia
-                    r="${c16_lidar_radius}"
-                    h="${c16_lidar_height}"
-                    mass="${c16_lidar_mass_kg}">
+                    r="${c16_radius}"
+                    h="${c16_height}"
+                    mass="${c16_mass_kg}">
                     <origin xyz="0 0 0" rpy="0 0 0" />
                 </xacro:cylinder_inertia>
@@ -71,14 +71,14 @@
             <xacro:if value="${model == 'c64'}">
                 <xacro:cylinder_inertia
-                    r="${c64_lidar_radius}"
-                    h="${c64_lidar_height}"
-                    mass="${c64_lidar_mass_kg}">
+                    r="${c64_radius}"
+                    h="${c64_height}"
+                    mass="${c64_mass_kg}">
                     <origin xyz="0 0 0" rpy="0 0 0" />
                 </xacro:cylinder_inertia>
             </xacro:if>
         </link>
-        <gazebo reference="${prefix}_${model}_lidar_link">
+        <gazebo reference="${prefix}_lslidar_${model}_lidar_link">
             <material>Gazebo/Blue</material>
-            <sensor name="${prefix}_${model}_lidar_sensor" type="ray">
+            <sensor name="${prefix}_lslidar_${model}_lidar_sensor" type="ray">
                 <pose>0 0 0.0 0 0 0</pose>
                 <visualize>true</visualize>
@@ -89,15 +89,15 @@
                             <xacro:if value="${model == 'c16'}">
                                 <samples>
-                                    ${(c16_lidar_horizontal_max_angle-c16_lidar_horizontal_min_angle)*(180/pi)/0.018/c16_lidar_hz}
+                                    ${(c16_horizontal_max_angle-c16_horizontal_min_angle)*(180/pi)/0.018/c16_hz}
                                 </samples>
-                                <min_angle>${c16_lidar_horizontal_min_angle}</min_angle>
-                                <max_angle>${c16_lidar_horizontal_max_angle}</max_angle>
+                                <min_angle>${c16_horizontal_min_angle}</min_angle>
+                                <max_angle>${c16_horizontal_max_angle}</max_angle>
                             </xacro:if>
                             <xacro:if value="${model == 'c64'}">
                                 <samples>
-                                    ${(c64_lidar_horizontal_max_angle-c64_lidar_horizontal_min_angle)*(180/pi)/0.018/c64_lidar_hz}
+                                    ${(c64_horizontal_max_angle-c64_horizontal_min_angle)*(180/pi)/0.018/c64_hz}
                                 </samples>
-                                <min_angle>${c64_lidar_horizontal_min_angle}</min_angle>
-                                <max_angle>${c64_lidar_horizontal_max_angle}</max_angle>
+                                <min_angle>${c64_horizontal_min_angle}</min_angle>
+                                <max_angle>${c64_horizontal_max_angle}</max_angle>
                             </xacro:if>
                         </horizontal>
@@ -105,12 +105,12 @@
                             <resolution>1</resolution>
                             <xacro:if value="${model == 'c16'}">
-                                <samples>${c16_lidar_number_of_channels}</samples>
-                                <min_angle>${c16_lidar_vertical_min_angle}</min_angle>
-                                <max_angle>${c16_lidar_vertical_max_angle}</max_angle>
+                                <samples>${c16_number_of_channels}</samples>
+                                <min_angle>${c16_vertical_min_angle}</min_angle>
+                                <max_angle>${c16_vertical_max_angle}</max_angle>
                             </xacro:if>
                             <xacro:if value="${model == 'c64'}">
-                                <samples>${c64_lidar_number_of_channels}</samples>
-                                <min_angle>${c64_lidar_vertical_min_angle}</min_angle>
-                                <max_angle>${c64_lidar_vertical_max_angle}</max_angle>
+                                <samples>${c64_number_of_channels}</samples>
+                                <min_angle>${c64_vertical_min_angle}</min_angle>
+                                <max_angle>${c64_vertical_max_angle}</max_angle>
                             </xacro:if>
                         </vertical>
@@ -118,10 +118,10 @@
                     <range>
                         <xacro:if value="${model == 'c16'}">
-                            <min>${c16_lidar_range_min}</min>
-                            <max>${c16_lidar_range_max}</max>
+                            <min>${c16_range_min}</min>
+                            <max>${c16_range_max}</max>
                         </xacro:if>
                         <xacro:if value="${model == 'c64'}">
-                            <min>${c64_lidar_range_min}</min>
-                            <max>${c64_lidar_range_max}</max>
+                            <min>${c64_range_min}</min>
+                            <max>${c64_range_max}</max>
                         </xacro:if>
                     </range>
@@ -129,13 +129,13 @@
                 <plugin name="gazebo_ros_block_laser" filename="libgazebo_ros_block_laser.so">
                     <robotNamespace>/</robotNamespace>
-                    <frameName>${prefix}_${model}_lidar_link</frameName>
-                    <topicName>${prefix}_${model}_lidar_points</topicName>
+                    <frameName>${prefix}_lslidar_${model}_lidar_link</frameName>
+                    <topicName>${prefix}_lslidar_${model}_lidar_point_cloud</topicName>
                     <gaussianNoise>0.01</gaussianNoise>
                     <hokuyoMinIntensity>101</hokuyoMinIntensity>
                     <xacro:if value="${model == 'c16'}">
-                        <updateRate>${c16_lidar_hz}</updateRate>
+                        <updateRate>${c16_hz}</updateRate>
                     </xacro:if>
                     <xacro:if value="${model == 'c64'}">
-                        <updateRate>${c64_lidar_hz}</updateRate>
+                        <updateRate>${c64_hz}</updateRate>
                     </xacro:if>
                 </plugin>

Commit message: returned the orientation of the imu frame back (as in a real sensor), reduced the gps frequency and removed the error for variables related to the Z axis

File: maddrive_urdf_tools/urdf/macros/gps.urdf.xacro (robot description, xacro)
@@ -36,5 +36,5 @@
         <gazebo>
             <plugin name="gazebo_ros_gps_sensor" filename="libhector_gazebo_ros_gps.so">
-                <updateRate>4.0</updateRate>
+                <updateRate>1.0</updateRate>
                 <robotNamespace>/</robotNamespace>
                 <bodyName>${prefix}_gps_sensor_link</bodyName>
@@ -49,11 +49,11 @@
                 <!-- <service>10</service> -->
                 <offset>0.0 0.0 0.0</offset>
-                <drift>0.001 0.001 0.001</drift>
-                <driftFrequency>0.001 0.001 0.001</driftFrequency>
-                <gaussianNoise>0.05 0.05 0.05</gaussianNoise>
-                <velocityOffset>0.001 0.001 0.001</velocityOffset>
-                <velocityDrift>0.001 0.001 0.001</velocityDrift>
-                <velocityDriftFrequency>0.001 0.001 0.001</velocityDriftFrequency>
-                <velocityGaussianNoise>0.5 0.5 0.5</velocityGaussianNoise>
+                <drift>0.001 0.001 0.0</drift>
+                <driftFrequency>0.001 0.001 0.0</driftFrequency>
+                <gaussianNoise>0.05 0.05 0.0</gaussianNoise>
+                <velocityOffset>0.001 0.001 0.0</velocityOffset>
+                <velocityDrift>0.001 0.001 0.0</velocityDrift>
+                <velocityDriftFrequency>0.001 0.001 0.0</velocityDriftFrequency>
+                <velocityGaussianNoise>0.5 0.5 0.0</velocityGaussianNoise>
             </plugin>
         </gazebo>

File: maddrive_urdf_tools/urdf/macros/realsense.urdf.xacro (robot description, xacro)
@@ -139,5 +139,5 @@
             <parent link="${prefix}_rs_${model}_camera_link" />
             <child link="${prefix}_rs_${model}_camera_imu_link" />
-            <origin xyz="0 0 0" rpy="${-pi/2} 0 ${-pi/2}" /> <!-- realsense2_description/launch/view_d435i(d455)_model.launch -->
+            <origin xyz="0 0 0" rpy="0 0 0" />
         </joint>
         <link name="${prefix}_rs_${model}_camera_imu_link">

File: maddrive_urdf_tools/urdf/macros/sector_lidar.urdf.xacro (robot description, xacro)
@@ -11,5 +11,5 @@
     <xacro:property name="c16_vertical_min_angle" value="-0.261799" />
     <xacro:property name="c16_vertical_max_angle" value="0.261799" />
-    <xacro:property name="c16_range_min" value="0.5" />
+    <xacro:property name="c16_range_min" value="2" />
     <xacro:property name="c16_range_max" value="150" />
     <xacro:property name="c64_mass_kg" value="1.0" />
