Commit message: little fixes in urdf macros

File: maddrive_urdf_tools/urdf/macros/gps.urdf.xacro (robot description, xacro)
@@ -2,19 +2,19 @@
 <robot xmlns:xacro="http://ros.org/wiki/xacro">
     <xacro:include filename="$(find maddrive_urdf_tools)/urdf/macros/inertia.urdf.xacro" />
-    <xacro:property name="gps_sensor_length" value="0.05" />
-    <xacro:property name="gps_sensor_width" value="0.05" />
-    <xacro:property name="gps_sensor_height" value="0.05" />
-    <xacro:property name="gps_sensor_mass" value="0.1" />
-    <xacro:macro name="gps_sensor" params="prefix parent origin_xyz origin_rpy">
-        <joint name="${prefix}_gps_sensor_joint" type="fixed">
+    <xacro:property name="ublox_gps_sensor_length" value="0.05" />
+    <xacro:property name="ublox_gps_sensor_width" value="0.05" />
+    <xacro:property name="ublox_gps_sensor_height" value="0.05" />
+    <xacro:property name="ublox_gps_sensor_mass" value="0.1" />
+    <xacro:macro name="ublox_gps_sensor" params="prefix parent origin_xyz origin_rpy">
+        <joint name="${prefix}_ublox_gps_sensor_joint" type="fixed">
             <parent link="${parent}" />
-            <child link="${prefix}_gps_sensor_link" />
+            <child link="${prefix}_ublox_gps_sensor_link" />
             <origin xyz="${origin_xyz}" rpy="${origin_rpy}" />
         </joint>
-        <link name="${prefix}_gps_sensor_link">
+        <link name="${prefix}_ublox_gps_sensor_link">
             <collision>
                 <origin xyz="0 0 0" rpy="0 0 0" />
                 <geometry>
-                    <box size="${gps_sensor_length} ${gps_sensor_width} ${gps_sensor_height}" />
+                    <box size="${ublox_gps_sensor_length} ${ublox_gps_sensor_width} ${ublox_gps_sensor_height}" />
                 </geometry>
             </collision>
@@ -22,12 +22,12 @@
                 <origin xyz="0 0 0" rpy="0 0 0" />
                 <geometry>
-                    <box size="${gps_sensor_length} ${gps_sensor_width} ${gps_sensor_height}" />
+                    <box size="${ublox_gps_sensor_length} ${ublox_gps_sensor_width} ${ublox_gps_sensor_height}" />
                 </geometry>
             </visual>
             <xacro:box_inertia
-                length="${gps_sensor_length}"
-                width="${gps_sensor_width}"
-                height="${gps_sensor_height}"
-                mass="${gps_sensor_mass}">
+                length="${ublox_gps_sensor_length}"
+                width="${ublox_gps_sensor_width}"
+                height="${ublox_gps_sensor_height}"
+                mass="${ublox_gps_sensor_mass}">
                 <origin xyz="0 0 0" rpy="0 0 0" />
             </xacro:box_inertia>
@@ -38,10 +38,10 @@
                 <updateRate>1.0</updateRate>
                 <robotNamespace>/</robotNamespace>
-                <bodyName>${prefix}_gps_sensor_link</bodyName>
-                <frameId>${prefix}_gps_sensor</frameId>
-                <topicName>${prefix}_gps_sensor/fix</topicName>
-                <velocityTopicName>${prefix}_gps_sensor/vel</velocityTopicName>
-                <referenceLatitude>0.0</referenceLatitude> <!-- широта -->
-                <referenceLongitude>0.0</referenceLongitude> <!-- долгота -->
+                <bodyName>${prefix}_ublox_gps_sensor_link</bodyName>
+                <frameId>${prefix}_ublox_gps_sensor</frameId>
+                <topicName>${prefix}_ublox_gps_sensor/fix</topicName>
+                <velocityTopicName>${prefix}_ublox_gps_sensor/vel</velocityTopicName>
+                <referenceLatitude>59.972814</referenceLatitude> <!-- широта -->
+                <referenceLongitude>30.322828</referenceLongitude> <!-- долгота -->
                 <referenceAltitude>0.0</referenceAltitude> <!-- высота -->
                 <referenceHeading>90.0</referenceHeading> <!-- угол 0 (ТЕТА) (в градусах) --> <!-- http://docs.ros.org/en/noetic/api/robot_localization/html/_images/figure2.png -->
@@ -51,5 +51,5 @@
                 <drift>0.0 0.0 0.0</drift>
                 <driftFrequency>0.0 0.0 0.0</driftFrequency>
-                <gaussianNoise>0.5 0.5 0.0</gaussianNoise> <!-- в метрах -->
+                <gaussianNoise>0.05 0.05 0.0</gaussianNoise> <!-- в метрах -->
                 <velocityOffset>0.0 0.0 0.0</velocityOffset>
                 <velocityDrift>0.0 0.0 0.0</velocityDrift>

File: maddrive_urdf_tools/urdf/macros/wheels.urdf.xacro (robot description, xacro)
@@ -34,5 +34,5 @@
 	</xacro:macro>
 	<!-- SPEED WHEEL -->
-	<xacro:macro name="speed_wheel" params="prefix parent suspension_origin_xyz ">
+	<xacro:macro name="speed_wheel" params="prefix parent suspension_origin_xyz suspension_height">
 		<joint name="${prefix}_suspension_joint" type="fixed">
 			<parent link="${parent}" />
